File: hardware/OPNhydro_r2/OPNhydro_r2.kicad_sch (KiCad schematic)
At the start: 149 parts, among them J1 MKDS, J2 MKDS, J3 BNC, J4 BNC, J5 BNC, M1 ESP32-C6-DEVKIT, M2 pH, M3 EC, M4 RTD, P1 MSTB_0.2", P10 KAS SF-12V, P11 KAS SF-12V, P12 KAS SF-12V, P2 PHR-4, P3 MC_0.2", P4 DC40-1250, P5 PHR-4, P6 MC_0.15", P7 PHR_2mm, P8 PHR_2mm, P9 PHR_2mm, SW1 FLOAT, SW2 FLOAT, T1 SI2301, T2 BT3904, T3 IRLR2905, T4 BT3904, T5 AO3400A, U1 TPS62933, U2 AZ1117-3.3, U3 ADM3260, U4 ADM3260, U5 TMC2209, U6 TMC2209, U7 TMC2209

Commit message: update
Parts:
- removed C1, C12, C14, C15, C17, C2, C21, C23, C26, C28, C29, C30, C31, C38, C39, C40, C41, C42, C43, C44, C45, C46, C5, C7, C8: 100nF, Coert-Vonk:CAP X7R 100nF ±10 25V 0805, symbol Coert-Vonk:CAP X7R 100nF ±10% 25V 0805
- removed C10, C11, C13, C25, C27, C4: 10μF, Coert-Vonk:CAP X7R 10μF ±10 16V 0805, symbol Coert-Vonk:CAP X7R 10μF ±10% 16V 0805
- removed C16, C18, C22, C24: 10nF, Coert-Vonk:CAP X7R 10nF ±10% 50V 0805, symbol Coert-Vonk:CAP X7R 10nF ±10% 50V 0805
- removed C19: 1000μF, Coert-Vonk:CAP ALUM 1000μF ±20 10V, symbol Coert-Vonk:CAP ALUM 1000μF ±20% 10V
- removed C20: 22μF, Coert-Vonk:CAP X7R 22μF ±10 10V 1206, symbol Coert-Vonk:CAP X7R 22μF ±10% 10V 1206
- removed C3: 2200μF, Coert-Vonk:CAP ALUM 2200μF ±20 25V RADIAL, symbol Coert-Vonk:CAP ALUM 2200μF ±20% 25V RADIAL
- removed C32, C33, C34: 2.2μF, Coert-Vonk:CAP X7R 2.2μF ±10 10V, symbol Coert-Vonk:CAP X7R 2.2μF ±10% 10V
- removed C35, C36, C37: 22nF, Coert-Vonk:CAP X7R 22nF ±10 50V 0805, symbol Coert-Vonk:CAP X7R 22nF ±10% 50V 0805
- removed C47, C48, C49: 100μF, Coert-Vonk:CAP ALUM 100μF ±20 25V, symbol Coert-Vonk:CAP ALUM 100μF ±20% 25V
- removed C6: 33nF, Coert-Vonk:CAP X7R 33nF ±10 25V 0805, symbol Coert-Vonk:CAP X7R 33nF ±10% 25V 0805
- removed C9: 47μF, Coert-Vonk:CAP X5R 47μF ±10 10V 1206, symbol Coert-Vonk:CAP X5R 47μF ±10% 10V 1206
- removed D1: 15V, Coert-Vonk:DIODE TVS 15VWM 24.4VC SMBJ15A DO214AA, symbol Coert-Vonk:DIODE TVS 15VWM 24.4VC SMBJ15A DO214AA
- removed DC1: 12V/6A, symbol Coert-Vonk:SUPPLY DC 12V 72W
- removed F1: 5A PTC, Coert-Vonk:FUSE RKEF500 PTC 60V 5A, symbol Coert-Vonk:FUSE 5A 60V PTC RKEF500
- removed H6, H7, H8: PH_2mm, Coert-Vonk:TERM BLK HDR 6POS PH 2mm, symbol Coert-Vonk:TERM BLK HDR 6POS PH 2mm
- removed L1: 5.6µH, Coert-Vonk:IND 5.6µH 3.5A 40mΩ, symbol Coert-Vonk:IND 5.6µH 3.5A 40mΩ
- removed P10, P11, P12: KAS SF-12V, symbol Coert-Vonk:PUMP KAMOER KAS SF-12V
- removed P4: DC40-1250, symbol Coert-Vonk:PUMP AUBIG DC40-1250
- removed P7, P8, P9: PHR_2mm, Coert-Vonk:TERM BLK PLG 6POS PHR 2mm, symbol Coert-Vonk:TERM BLK PLG 6POS PHR 2mm
- removed PR1: USS, symbol Coert-Vonk:PROBE ULTRASONIC SENSOR
- removed PR4: EC_K1.0, symbol Coert-Vonk:PROBE ATLAS ENV-40-EC-K1.0
- removed R1, R18, R2, R23, R25, R27, R9: 4k7, Coert-Vonk:RES 4.7kΩ ±1 18W Yageo 0805, symbol Coert-Vonk:RES 4.7kΩ ±1% 1/8W Yageo 0805
- removed R10, R12, R15, R16, R19, R3, R5, R7: 10k, Coert-Vonk:RES 10kΩ ±1 18W Yageo 0805, symbol Coert-Vonk:RES 10kΩ ±1% 1/8W Yageo 0805
- removed R11: 52k3, Coert-Vonk:RES 52.3kΩ 0805, symbol Coert-Vonk:RES 52.3kΩ ±1% 1/8W Yageo 0805
- removed R13, R14: 16k9, Coert-Vonk:RES 16.9kΩ ±1 18W 0805, symbol Coert-Vonk:RES 16.9kΩ ±1% 1/8W Yageo 0805
- removed R17, R20, R21, R22, R8: 100Ω, Coert-Vonk:RES 100Ω ±1 18W Yageo 0805, symbol Coert-Vonk:RES 100Ω ±1% 1/8W Yageo 0805
- removed R24, R26, R28, R6: 1k, Coert-Vonk:RES 1kΩ ±1 18W Yageo 0805, symbol Coert-Vonk:RES 1kΩ ±1% 1/8W Yageo 0805
- removed R29, R30, R31, R32, R33, R34: 220mΩ, Coert-Vonk:RES 220mΩ ±1 18W Yageo 0805, symbol Coert-Vonk:RES 220mΩ ±1% 1/4W Yageo 0805
- removed R4: 100k, Coert-Vonk:RES 100kΩ 0805, symbol Coert-Vonk:RES 100kΩ ±1% 1/8W Yageo 0805
- removed T1: SI2301, Coert-Vonk:MOSFET P-CH 20V 3.1A SI2301CDS SOT23-3, symbol Coert-Vonk:MOSFET P-CH 20V 3.1A SI2301 SOT23-3
- removed V1: 2V025-08, symbol Coert-Vonk:VALVE ANGGREK 2V025-08
- added C1, C11, C15, C17, C19, C2, C21, C25, C27, C30, C32, C33, C34, C35, C42, C43, C44, C45, C46, C47, C48, C49, C5, C50, C54, C7, C8: 100nF, Coert-Vonk:CAP X7R 100nF ±10 50V 0402 Murata, symbol Coert-Vonk:CAP X7R 100nF ±10% 50V 0402 Murata
- added C10, C12, C13, C14, C16, C18, C29, C31: 10μF, Coert-Vonk:CAP X5R 10μF ±10 16V 0805 Murata GRM, symbol Coert-Vonk:CAP X5R 10μF ±10% 16V 0805 Murata GRM
- added C20, C22, C26, C28: 10nF, Coert-Vonk:CAP X7R 10nF ±10 16V 0402 Murata, symbol Coert-Vonk:CAP X7R 10nF ±10% 16V 0402 Murata
- added C23: 220μF, Coert-Vonk:CAP ALUM-POLY 220μF ±20 16V Panasonic, symbol Coert-Vonk:CAP ALUM-POLY 220μF ±20% 16V Panasonic
- added C24: 22μF, Coert-Vonk:CAP X7R 22μF ±10 10V 1206, symbol Coert-Vonk:CAP X7R 22μF ±10% 10V 1206 Murata GRM
- added C3: 1000μF, Coert-Vonk:CAP ALUM 1000μF ±20 50V Panasonic, symbol Coert-Vonk:CAP ALUM-ELEC 1000μF ±20% 50V Panasonic
- added C36, C37, C38: 2.2μF, Coert-Vonk:CAP X7R 2.2μF ±10 10V 0603 Murata, symbol Coert-Vonk:CAP X7R 2.2μF ±10% 10V 0603 Murata
- added C39, C40, C41: 22nF, Coert-Vonk:CAP X7R 22nF ±10 100V 0603 Murata, symbol Coert-Vonk:CAP X7R 22nF ±10% 100V 0603 Murata
- added C4: 10μF, Coert-Vonk:CAP X7R 10μF ±10 50V 1206 Murata GRT, symbol Coert-Vonk:CAP X7R 10μF ±10% 50V 1206 Murata GRT
- added C51, C52, C53: 220μF/50V, Coert-Vonk:CAP ALUM 220μF ±20 50V Panasonic, symbol Coert-Vonk:CAP ALUM-ELEC 220μF ±20% 50V Panasonic
- added C6: 33nF, Coert-Vonk:CAP X7R 33nF ±10 50V 0805 Kemet, symbol Coert-Vonk:CAP X7R 33nF ±10% 50V 0805 Kemet
- added C9: 470μF/50V, Coert-Vonk:CAP ALUM 470μF ±20 50V Panasonic, symbol Coert-Vonk:CAP ALUM-ELEC 470μF ±20% 50V Panasonic
- added D1: 28V, Coert-Vonk:DO-214AA, symbol Coert-Vonk:DIODE TVS 30VWM 48.4VC SMCJ30A DO-214AA
- added D4: 12V, Coert-Vonk:SOD323_DIO, symbol Coert-Vonk:DIODE ZENER 12V 200mW SOD-323 Diodes
- added DC1: 24V/6.5A, symbol Coert-Vonk:SUPPLY DC 24V 156W
- added F1: 7A, Coert-Vonk:FUSE 2-SMD, symbol Coert-Vonk:FUSE 7A 125V 2-SMD
- added FB1: 50Ω@100Mhz/12A, Coert-Vonk:FERRITE BEAD 12A 1.6mΩ 50Ω 1206 Murata, symbol Coert-Vonk:FERRITE BEAD 12A 1.6mΩ 50Ω 1206 Murata
- added H6, H7, H8: JST_XH, Coert-Vonk:TERM BLK HDR 4POS JST-XH 2.5mm, symbol Coert-Vonk:TERM BLK HDR 4POS JST-XH 2.5mm
- added L1: 10µH, Coert-Vonk:IND 10µH 5.6A 21mΩ, symbol Coert-Vonk:IND 10µH 5.6A 21mΩ
- added P10, P11, P12: ANKO_A200SX, symbol Coert-Vonk:PUMP ANKO A200SX
- added P13, P14, P15: XH_2.5mm, Coert-Vonk:TERM BLK PLG 4POS XH 2.5mm, symbol Coert-Vonk:TERM BLK PLG 4POS JST-XH 2.5mm
- added P4: DC40F-2460, symbol Coert-Vonk:PUMP SHYSKY DC40F-2460
- added PR1: LiDAR, symbol Coert-Vonk:PROBE LiDAR BENEWAKE TF-LUNA
- added PR4: BL_EC, symbol Coert-Vonk:PROBE BLUELAB PROBPCEC
- added R1, R19, R2, R21, R26, R28: 4k7, Coert-Vonk:RES 0805 YAGEO, symbol Coert-Vonk:RES 4.7kΩ ±1% 1/8W 0805 Yageo
- added R10, R18, R20, R22, R23, R9: 100Ω, Coert-Vonk:RES 100Ω ±1 18W Yageo 0805, symbol Coert-Vonk:RES 100Ω ±1% 1/8W 0805 Yageo
- added R11, R12, R15, R16, R17, R3, R7: 10k, Coert-Vonk:RES 0805 YAGEO, symbol Coert-Vonk:RES 10kΩ ±1% 1/8W 0805 Yageo
- added R13, R14: 16k9, Coert-Vonk:RES 0805 YAGEO, symbol Coert-Vonk:RES 16.9kΩ ±1% 1/8W 0805 Yageo
- added R24, R27, R29, R6: 1k, Coert-Vonk:RES 0805 YAGEO, symbol Coert-Vonk:RES 1kΩ ±1% 1/8W 0805 Yageo
- added R25, R30, R31, R32, R33, R34: 220mΩ, Coert-Vonk:RES 0805 YAGEO, symbol Coert-Vonk:RES 220mΩ ±1% 1/4W 0805 Yageo
- added R4: 33k, Coert-Vonk:RES 0805 YAGEO, symbol Coert-Vonk:RES 33kΩ ±1% 1/8W 0805 Yageo
- added R5: 52k3, Coert-Vonk:RES 0805 YAGEO, symbol Coert-Vonk:RES 52.3kΩ ±1% 1/8W 0805 Yageo
- added R8: 21k, Coert-Vonk:RES 0805 YAGEO, symbol Coert-Vonk:RES 21kΩ ±1% 1/8W 0805 Yageo
- added T1: AON6407, Coert-Vonk:MOSFET P-CH 30V 32A 10mΩ AON6407, symbol Coert-Vonk:MOSFET P-CH 30V 32A 10mΩ AON6407
- added V1: DIGITEN-24V, symbol Coert-Vonk:VALVE DIGITEN DC 24V 1/4{dblquote} NC COMIN16JU031071
- M2: value pH -> ATLAS_EZO_pH
- M3: value EC -> ATLAS_EZO_EC
- M4: value RTD -> ATLAS_EZO_RTD
- PR3: value pH -> BL_pH; symbol Coert-Vonk:PROBE ATLAS ENV-40-PH -> Coert-Vonk:PROBE BLUELAB PROBPH; BLPN (none) -> PROBPH
- PR5: value RTD -> ATLAS_RTD
- renumbered FB1 to FB2, FB2 to FB3, FB3 to FB4, FB4 to FB5
Connections:
- net 0V8: now also R12.2, R5.1
- net 3V3: now also C11.2, C12.2, C2.2, C24.2, C25.2, C26.1, C27.2, C28.1, C29.2, C30.1, C31.2, C32.1, C33.2, C34.2, C35.2, R1.2, R2.2, R21.2, R26.2, R28.2, R3.2
- net 5V: now also C10.2, C13.2, C18.2, C23.1, L1.2, R5.2
- net ATO_VALVE: now also R18.1
- net FLOAT_HIGH: now also C2.1, R10.1, R7.2
- net FLOAT_LOW: now also C1.2, R19.1, R3.1
- net GND: now also C1.1, C10.1, C11.1, C12.1, C13.1, C18.1, C23.2, C24.1, C25.1, C26.2, C27.1, C28.2, C29.1, C3.2, C30.2, C31.1, C32.2, C33.1, C34.1, C35.1, C36.1, C37.1, C38.1, C4.1, C45.1, C46.1, C47.1, C48.1, C49.1, C5.1, C50.1, C51.2, C52.2, C53.2, C54.1, C6.1, C7.1, C9.2, D1.2 (A), D4.2 (A), R11.1, R12.1, R17.1, R24.1, R25.2, R27.1, R29.1, R30.2, R31.2, R32.2, R33.2, R34.2, R7.1, R8.1; no longer U5.2 (~{EN}), U6.2 (~{EN}), U7.2 (~{EN})
- net I2C_SCL: now also J1.3 (Pin_3), R1.1
- net I2C_SDA: now also J1.2 (Pin_2), R2.1
- net PUMP_MAIN: now also R9.1
- net STEP_BUS: now also R20.1, R22.1, R23.1, R6.2
- net at U7.23 (BRA): now also R33.1
- net at FB4.1, FB5.1, M3.1 (GND)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: now also C17.1, C22.1, R13.2
- net at U4.13 (VSEL): now also R13.1, R15.1
- net at T2.1 (B): now also R10.2
- net at U5.8 (5VOUT): now also C36.2
- net at FB4.2, U4.12 (V_{ISO}): now also C16.2, C21.2
- net at D2.A, H3.2, T3.3 (D): now also C7.2, C9.1
- net at U6.4 (CPO): now also C40.1
- net at U6.5 (CPI): now also C40.2
- net at U7.8 (5VOUT): now also C38.2
- net at U1.5 (SW): now also C8.2, L1.1
- net at U7.4 (CPO): now also C41.1
- net at U7.5 (CPI): now also C41.2
- net at T4.1 (B): now also R19.2
- net at FB5.2, U4.11 (GND_{ISO}), U4.14 (GND_{ISO})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: now also C16.1, C17.2, C21.1, C22.2, R15.2
- net at U5.14 (~{PD}/UART): now also R20.2
- net at FB2.1, FB3.1, M2.1 (GND)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: now also C15.1, C20.1, R14.2
- net at FB2.2, U3.12 (V_{ISO}): now also C14.2, C19.2
- net at U5.17 (VREF): now also R21.1, R24.2
- net at T4.3 (C), T5.1 (G): now also R17.2, R18.2
- net at D3.A, H5.2, T5.3 (D): now also C54.2
- net at FB3.2, U3.11 (GND_{ISO}), U3.14 (GND_{ISO})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: now also C14.1, C15.2, C19.1, C20.2, R16.2
- net at U7.1 (OB2): now also H8.4
- net at U7.14 (~{PD}/UART): now also R23.2
- net at U7.17 (VREF): now also R28.1, R29.2
- net at U7.21 (OA2): now also H8.2
- net at U7.24 (OA1): now also H8.1
- net at U7.26 (OB1): now also H8.3
- net at U7.27 (BRB): now also R34.1
- net at U7.6 (VCP): now also C44.1
- net at U5.1 (OB2): now also H6.4
- net at U5.21 (OA2): now also H6.2
- net at U5.23 (BRA): now also R25.1
- net at U5.24 (OA1): now also H6.1
- net at U5.26 (OB1): now also H6.3
- net at U5.27 (BRB): now also R30.1
- net at U5.4 (CPO): now also C39.1
- net at U5.5 (CPI): now also C39.2
- net at U5.6 (VCP): now also C42.1
- net at T2.3 (C), T3.1 (G): now also R11.2, R9.2
- net at U6.27 (BRB): now also R32.1
- net at P6.1: now also V1.24V
- net at P6.2: now also V1.GND
- net at U6.1 (OB2): now also H7.4
- net at U6.14 (~{PD}/UART): now also R22.2
- net at U6.17 (VREF): now also R26.1, R27.2
- net at U6.21 (OA2): now also H7.2
- net at U6.23 (BRA): now also R31.1
- net at U6.24 (OA1): now also H7.1
- net at U6.26 (OB1): now also H7.3
- net at U6.6 (VCP): now also C43.1
- net at U6.8 (5VOUT): now also C37.2
- net at P1.1: now also DC1.24V
- net at P1.2: now also DC1.GND
- net at H1.1: now also FB1.1
- net at U3.13 (VSEL): now also R14.1, R16.1
- net at U1.7 (SS): now also C6.2
- net at U1.6 (BST): now also C8.1
- net at P3.1: now also P4.24V
- net at P3.2: now also P4.GND
- net at M1.J3_6 (TX1/IO22): now also R6.1
- net STEP_PDIS: now reaches M1.J3_8 (IO20)
- net STEP_PDIS: now also U5.2 (~{EN}), U6.2 (~{EN}), U7.2 (~{EN})
- net at U1.1 (RT): now also R8.2
- net 12V renamed 24V
- net 24V: now also C3.1, C4.2, C42.2, C43.2, C44.2, C45.2, C46.2, C47.2, C48.2, C49.2, C5.2, C50.2, C51.1, C52.1, C53.1, T1.3 (D)
- net US_ECHO: no longer names the net of M1.J1_13 (IO3/ADC3)
- net US_ECHO: no longer J1.3 (Pin_3)
- net US_TRIG: no longer names the net of M1.J1_6 (IO7/SPI_MOSI)
- net US_TRIG: no longer J1.2 (Pin_2)
- new net: P11.1 (A1), P14.1
- new net: P11.2 (A2), P14.2
- new net: P11.3 (B1), P14.3
- new net: P11.4 (B2), P14.4
- new net: P12.1 (A1), P15.1
- new net: P12.2 (A2), P15.2
- new net: P12.3 (B1), P15.3
- new net: P12.4 (B2), P15.4
- new net: F1.1, FB1.2
- new net: D1.1 (C), F1.2, R4.2, T1.2 (S)
- new net: D4.1 (K), R4.1, T1.1 (G)
- new net: P10.1 (A1), P13.1
- new net: P10.2 (A2), P13.2
- new net: P10.3 (B1), P13.3
- new net: P10.4 (B2), P13.4
Other:
- note added: "24V→5V 3A BUCK"
- note added: "bulk for WiFi Tx"
- note added: "bulk for simultaneous motors"
- note added: "f_{SW}=1MHz"
- note added: "t_{ss}=5ms"
- note removed: "12V→5V 3A BUCK"
- note removed: "5ms soft-start"
- note removed: "Bootstrap"
- note removed: "Bulk for motor surge"
- note removed: "Bulk for radio TX"
- moved on the sheet: D2, H3, M1B, P3, T2, T3, T4, U1, U2

Commit message: update
Parts:
- removed C9: 470μF/50V, Coert-Vonk:CAP ALUM 470μF ±20 50V Panasonic, symbol Coert-Vonk:CAP ALUM-ELEC 470μF ±20% 50V Panasonic
- removed R1, R2: 4k7, Coert-Vonk:RES 0805 YAGEO, symbol Coert-Vonk:RES 4.7kΩ ±1% 1/8W 0805 Yageo
- added C11: 220μF/50V, Coert-Vonk:CAP ALUM 220μF ±20 50V Panasonic, symbol Coert-Vonk:CAP ALUM-ELEC 220μF ±20% 50V Panasonic
- added R1, R13, R14, R15, R16, R2: 2k2, Coert-Vonk:RES 0805 YAGEO, symbol Coert-Vonk:RES 2.2kΩ ±1% 1/8W 0805 Yageo
- renumbered C54 to C29, C29 to C30, C30 to C31, C31 to C32, C32 to C33, C33 to C34, C34 to C35, C35 to C36, C36 to C37, C37 to C38, C38 to C39, C39 to C40, C40 to C41, C41 to C42, C42 to C43, C43 to C44, C44 to C45, C45 to C46, C46 to C47, C47 to C48, C48 to C49, C49 to C50, C50 to C51, C53 to C52, C52 to C53, C51 to C54, C8 to C7, C7 to C8, C11 to C9, D4 to D2, D2 to D3, D3 to D4, P13 to P7, P14 to P8, P15 to P9, R11 to R10, R5 to R11, R14 to R17, R13 to R18, R16 to R19, R15 to R20, R18 to R21, R19 to R22, R17 to R23, R20 to R24, R22 to R25, R23 to R26, R21 to R27, R24 to R28, R26 to R29, R27 to R30, R28 to R31, R29 to R32, R25 to R33, R30 to R34, R31 to R35, R32 to R36, R33 to R37, R34 to R38, R6 to R5, R7 to R6, R8 to R7, R9 to R8, R10 to R9
Connections:
- net 3V3: now also R1.2, R2.2
- net GND: now also C11.2
- net I2C_SCL: now also R2.1
- net I2C_SDA: now also R1.1
- net V_{ISO,EC}: now reaches C17.1, C22.1, FB4.1, M3.6 (VCC), R18.2, U4.17 (VDD_{ISO})
- net V_{ISO,EC}: now also R14.2, R16.2; no longer FB5.1, M3.1 (GND)
- net at M3.2 (TX/SCL), U4.19 (SCL_{1}): now also R16.1
- net at M3.3 (RX/SDA), U4.18 (SDA_{1}): now also R14.1
- net at C8.2, D3.A, H3.2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: now also C11.1
- net V_{ISO,pH}: now reaches C15.1, C20.1, FB2.1, M2.6 (VCC), R17.2, U3.17 (VDD_{ISO})
- net V_{ISO,pH}: now also R13.2, R15.2; no longer FB3.1, M2.1 (GND)
- net at M2.2 (TX/SCL), U3.19 (SCL_{1}): now also R15.1
- net at M2.3 (RX/SDA), U3.18 (SDA_{1}): now also R13.1
- new net: FB5.1, M3.1 (GND)
- new net: FB3.1, M2.1 (GND)
Other:
- moved on the sheet: C14, C15, C16, C17, C19, C20, C21, C22, C25, C26, C27, C28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

Commit message: update
Parts:
- removed FB2, FB3, FB4, FB5: 330Ω at 100MHz, Coert-Vonk:FERRITE BEAD 330Ω 0805, symbol Coert-Vonk:FERRITE BEAD 330Ω 0805
- added C1: 100μF, Coert-Vonk:CAP ALUM 100μF ±20 25V, symbol Coert-Vonk:CAP ALUM-ELEC 100μF ±20% 25V Panasonic
- added FB2, FB3, FB4, FB5: 60Ω at 100MHz, symbol Coert-Vonk:FERRITE BEAD 20mΩ 60Ω 0603 TDK
- C21: renamed from C20; PN (none) -> GRM155R71C103KA01D
- renumbered C9 to C10, C10 to C11, C11 to C12, C12 to C13, C13 to C14, C14 to C15, C15 to C16, C16 to C17, C17 to C18, C18 to C19, C1 to C2, C19 to C20, C21 to C22, C22 to C23, C23 to C24, C24 to C25, C25 to C26, C26 to C27, C27 to C28, C28 to C29, C2 to C3, C29 to C30, C30 to C31, C31 to C32, C32 to C33, C33 to C34, C34 to C35, C35 to C36, C36 to C37, C37 to C38, C38 to C39, C3 to C4, C39 to C40, C40 to C41, C41 to C42, C42 to C43, C43 to C44, C44 to C45, C45 to C46, C46 to C47, C47 to C48, C48 to C49, C4 to C5, C49 to C50, C50 to C51, C51 to C52, C52 to C53, C53 to C54, C54 to C55, C5 to C6, C6 to C7, C7 to C8, C8 to C9
Connections:
- net 3V3: now also C1.1
- net GND: now also C1.2
- net V_{ISO,EC}: now also FB4.1
- net V_{ISO,pH}: now also FB2.1
- net at M3.1 (GND): now also FB5.1
- net at C17.2, C22.2, U4.12 (V_{ISO}): now also FB4.2
- net at C17.1, C18.2, C22.1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: now also FB5.2
- net at C15.2, C20.2, U3.12 (V_{ISO}): now also FB2.2
- net at M2.1 (GND): now also FB3.1
- net at C15.1, C16.2, C20.1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: now also FB3.2
Other:
- moved on the sheet: C10, C11, C12, C13, C14, C15, C16, C17, C18, C19, C2, C20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

Commit message: update
Parts:
- removed C36, C37: 100nF, Coert-Vonk:CAP X7R 100nF ±10 50V 0402 Murata, symbol Coert-Vonk:CAP X7R 100nF ±10% 50V 0402 Murata
- removed C39, C40: 2.2μF, Coert-Vonk:CAP X7R 2.2μF ±10 10V 0603 Murata, symbol Coert-Vonk:CAP X7R 2.2μF ±10% 10V 0603 Murata
- removed R24, R25, R26: 100Ω, Coert-Vonk:RES 100Ω ±1 18W Yageo 0805, symbol Coert-Vonk:RES 100Ω ±1% 1/8W 0805 Yageo
- removed R27, R29, R31: 4k7, Coert-Vonk:RES 0805 YAGEO, symbol Coert-Vonk:RES 4.7kΩ ±1% 1/8W 0805 Yageo
- removed R28, R30, R32: 1k, Coert-Vonk:RES 0805 YAGEO, symbol Coert-Vonk:RES 1kΩ ±1% 1/8W 0805 Yageo
- removed R34, R35, R36, R37, R38: 220mΩ, Coert-Vonk:RES 0805 YAGEO, symbol Coert-Vonk:RES 220mΩ ±1% 1/4W 0805 Yageo
- added C36, C37: 2.2μF, Coert-Vonk:CAP X7R 2.2μF ±10 10V 0603 Murata, symbol Coert-Vonk:CAP X7R 2.2μF ±10% 10V 0603 Murata
- added C39, C40: 100nF, Coert-Vonk:CAP X7R 100nF ±10 50V 0402 Murata, symbol Coert-Vonk:CAP X7R 100nF ±10% 50V 0402 Murata
- added R24, R25, R26, R34, R35: 110mΩ, Coert-Vonk:RES 0805 YAGEO, symbol Coert-Vonk:RES 110mΩ ±1% 1/8W 0805 Susumu
- added R27, R29, R31: 14k, Coert-Vonk:RES 0805 YAGEO, symbol Coert-Vonk:RES 14kΩ ±1% 1/8W 0805 Yageo
- added R28, R30, R32: 10k7, Coert-Vonk:RES 0805 YAGEO, symbol Coert-Vonk:RES 10.7kΩ ±1% 1/8W 0805 Yageo
- R33: value 220mΩ -> 110mΩ; symbol Coert-Vonk:RES 220mΩ ±1% 1/4W 0805 Yageo -> Coert-Vonk:RES 110mΩ ±1% 1/8W 0805 Susumu; DKPN 311-0.22LUCT-ND -> RL12S.11FCT-ND
Connections:
- net 3V3: now also U6.10 (MS2/AD1), U7.9 (MS1/AD0), C39.2, C40.2; no longer U5.19 (DIR), U6.19 (DIR), U6.9 (MS1/AD0), U7.19 (DIR)
- net GND: now also C36.1, C37.1, C39.1, C40.1, R24.2, R25.2, R26.2, R28.1, R30.1, R32.1, R34.2, R35.2; no longer U5.10 (MS2/AD1), U5.9 (MS1/AD0), U6.10 (MS2/AD1), U7.9 (MS1/AD0)
- net STEP_BUS: now also U5.14 (~{PD}/UART), U6.14 (~{PD}/UART), U7.14 (~{PD}/UART)
- net at C38.2, U5.8 (5VOUT): now also R27.2
- net at U7.23 (BRA): now also R34.1
- net at U6.17 (VREF): now also R29.1, R30.2
- net at U7.17 (VREF): now also R31.1, R32.2
- net at U7.27 (BRB): now also R35.1
- net at U7.8 (5VOUT): now also C37.2, R31.2
- net at U5.17 (VREF): now also R27.1, R28.2
- net at U5.27 (BRB): now also R24.1
- net at U6.27 (BRB): now also R26.1
- net at U6.23 (BRA): now also R25.1
- net at U6.8 (5VOUT): now also C36.2, R29.2
- no-connect marks 25 -> 31
Other:
- note added: "addr=00"
- note added: "addr=10"
- note added: "addr=11"
- moved on the sheet: C35, C38, C41, C44, C47, C50, C53, H6, H7, P10, P11, P12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

Commit message: update
Parts:
- removed J1: MKDS, Coert-Vonk:TERM BLK 4POS SCREW 3.5mm, symbol Coert-Vonk:TERM BLK SCREW 4POS MKDS 3.5mm
- removed PR2: LIGHT, symbol Coert-Vonk:PROBE_LIGHT
- removed R9: 100Ω, Coert-Vonk:RES 100Ω ±1 18W Yageo 0805, symbol Coert-Vonk:RES 100Ω ±1% 1/8W 0805 Yageo
- added C56, C58: 100nF, Coert-Vonk:CAP X7R 100nF ±10 50V 0402 Murata, symbol Coert-Vonk:CAP X7R 100nF ±10% 50V 0402 Murata
- added C57, C59: 10μF, Coert-Vonk:CAP X5R 10μF ±10 16V 0805 Murata GRM, symbol Coert-Vonk:CAP X5R 10μF ±10% 16V 0805 Murata GRM
- added H9: PB_1.25mm, Coert-Vonk:TERM BLK HDR 6POS PB 1.25mm Molex, symbol Coert-Vonk:TERM BLK HDR 6POS MOLEX-PB 1.25mm
- added P13: PB_1.25mm, Coert-Vonk:TERM BLK PLG 6POS MOLEX-PB 1.25mm, symbol Coert-Vonk:TERM BLK PLG 6POS MOLEX-PB 1.25mm
- added PR2: LIGHT, symbol Coert-Vonk:PROBE LIGHT
- added R9: 4k7, Coert-Vonk:RES 0805 YAGEO, symbol Coert-Vonk:RES 4.7kΩ ±1% 1/8W 0805 Yageo
- H1: MFR (none) -> Phoenix Connect; MPN (none) -> 1757242
- H2, H4: MFR (none) -> JST; PN (none) -> S4B-PH-K-S
- H3: MFR (none) -> Phoenix Connect; MPN (none) -> 1836189
- H5: MFR (none) -> Phoenix Connect; MPN (none) -> 1803277
- J2: MFR (none) -> Phoenix Contact; MPN (none) -> 1751264
- P1: MFR (none) -> Phoenix Connect; MPN (none) -> 1757019
- P2, P5: value PHR-4 -> PHR_4
- P3: MFR (none) -> Phoenix Connect; MPN (none) -> 1836079
- P6: MFR (none) -> Phoenix Connect; MPN (none) -> 1803578
Connections:
- net 3V3: now also R10.2, C56.2, C57.2, C58.2, C59.2, H9.1
- net FLOAT_HIGH: now also R22.1
- net FLOAT_LOW: now also R9.1; no longer R22.1
- net GND: now also C56.1, C57.1, C58.1, C59.1, H9.4, H9.5, H9.S, H9.S2; no longer R10.1
- net I2C_SCL: now also H2.3 (SCL), H4.3 (SCL), H9.3; no longer H2.4 (I2C_SCL), H4.4 (I2C_SCL)
- net I2C_SDA: now also H2.4 (SDA), H4.4 (SDA), H9.2; no longer H2.3 (I2C_SDA), H4.3 (I2C_SDA)
- net GND_PUMP_MAIN: now reaches C12.1, C9.2, D3.A, H3.2, T3.3 (D)
- net at P2.1: now also PR2.1 (GND)
- net at P2.2: now also PR2.2 (VCC)
- net at P2.3: now also PR2.3 (SCL)
- net at P2.4: now also PR2.4 (SDA)
- net GND_ATO_VALVE: now reaches C30.2, D4.A, H5.2, T5.3 (D)
- net at R8.2, T2.3 (C), T3.1 (G): now also R10.1; no longer R10.2
- net at PR1.1 (VCC): now also P13.1
- net at PR1.2 (SDA): now also P13.2
- net at PR1.3 (SCL): now also P13.3
- net at PR1.4 (RDY): now also P13.6
- net at T2.1 (B): now also R9.2
- new net: P13.4, PR1.4 (RDY)
- new net: P13.5, PR1.4 (RDY)
- no-connect marks 31 -> 32
Other:
- note removed: "Flyback"
- note removed: "Prevent high-frequency oscillation"
- note removed: "Stay off during SoC reset"
- moved on the sheet: C1, C12, C2, C3, C30, C9, J2, P2, P5, R10, R21, R22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

Commit message: update
Parts:
- removed C30: 100nF, Coert-Vonk:CAP X7R 100nF ±10 50V 0402 Murata, symbol Coert-Vonk:CAP X7R 100nF ±10% 50V 0402 Murata
- added C30: 47μF, Coert-Vonk:CAP ALUM-ELEC 47μF ±20 50V Panasonic, symbol Coert-Vonk:CAP ALUM-ELEC 47μF ±20% 50V Panasonic
- added C61: 100nF, Coert-Vonk:CAP X7R 100nF ±10 50V 0402 Murata, symbol Coert-Vonk:CAP X7R 100nF ±10% 50V 0402 Murata
Connections:
- net 24V: now also C12.1, C9.2, C30.1, C61.2
- net 3V3: no longer C1.1, H9.1
- net 5V: now also C1.1, H9.1
- net GND: now also C30.2, C61.1
- net GND_ATO_VALVE: no longer names the net of D4.A, H5.2, T5.3 (D)
- net GND_PUMP_MAIN: no longer names the net of D3.A, H3.2, T3.3 (D)
- net GND_PUMP_MAIN: no longer C12.1, C9.2
Other:
- moved on the sheet: C12, C9, R10, R21, R22, R23, R8, R9, T2, T3, T4, T5

Commit message: update
Parts:
- C11: MFR (none) -> Murata; PN (none) -> GRM21BR61C106KE15L
- C12: value 220μF/50V -> 220μF; MFR (none) -> Panasonic; PN (none) -> ECA-1HM221B; Series (none) -> M-A
- C15: MFR (none) -> Murata; PN (none) -> GRM21BR61C106KE15L; SERIES (none) -> GRM
- C24: MFR (none) -> Panasonic; PN (none) -> 16SVPK220M
- C5: MFR (none) -> Murata; PN (none) -> GRT31CR61H106KE01L
- C7: DKPN 399-C0805C333K5RACTUCT-ND -> 490-GRM155R71H333KE14JCT-ND; MFR (none) -> Murata; PN (none) -> GRM155R71H333KE14J
- C8: MFR (none) -> Murata; PN (none) -> GRM155R71H104KE14D
- FB2: MPN MPZ1608S600ATDH5 -> (none); PN (none) -> MPZ1608S600ATDH5; SERIES (none) -> MPZ
- R10: MFR (none) -> Yageo; PN (none) -> RC0805FR-0710KL; SERIES (none) -> RC_L
- R13: MFR (none) -> Yageo; SERIES (none) -> RC_L
- R7: MFR (none) -> Yageo; PN (none) -> RC0805FR-0721KL
- R8: DKPN 100 Ohms ±1% 0.125W, 1/8W Chip Resistor 0805 (2012 Metric) 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 -> (none); MFR (none) -> Yageo
- T2: MFR (none) -> Onsemi; PN (none) -> MMBT3904LT1G
- U1: MFR (none) -> Texas Instruments; PN (none) -> TPS62933DRLR
- U2: MFR (none) -> Diodes; PN (none) -> AZ1117IH-3.3TRG1
- U3: MFR (none) -> Analog Devices; PN (none) -> ADM3260ARSZ; SERIES (none) -> IsoPower

Commit message: update
Changed lines of the file:
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@@
 	)
 	(junction
-		(at 161.29 195.58)
-		(diameter 0)
-		(color 0 0 0 0)
-	)
-	(junction
 		(at 290.83 212.09)
 		(diameter 0)
@@
 	)
 	(junction
+		(at 167.64 195.58)
+		(diameter 0)
+		(color 0 0 0 0)
+	)
+	(junction
 		(at 173.99 195.58)
 		(diameter 0)
@@
 	)
 	(junction
-		(at 161.29 198.12)
-		(diameter 0)
-		(color 0 0 0 0)
-	)
-	(junction
-		(at 161.29 200.66)
-		(diameter 0)
-		(color 0 0 0 0)
-	)
-	(junction
 		(at 189.23 95.25)
 		(diameter 0)
@@
 	)
 	(junction
-		(at 167.64 195.58)
-		(diameter 0)
-		(color 0 0 0 0)
-	)
-	(junction
 		(at 171.45 38.1)
 		(diameter 0)
@@
 	(wire
 		(pts
-			(xy 158.75 195.58) (xy 161.29 195.58)
-		)
-		(stroke
-			(width 0)
-			(type default)
-		)
-	)
-	(wire
-		(pts
 			(xy 233.68 105.41) (xy 238.76 105.41)
 		)
@@
 	(wire
 		(pts
+			(xy 161.29 198.12) (xy 166.37 198.12)
+		)
+		(stroke
+			(width 0)
+			(type default)
+		)
+	)
+	(wire
+		(pts
 			(xy 290.83 223.52) (xy 290.83 222.25)
 		)
@@
 	(wire
 		(pts
+			(xy 161.29 195.58) (xy 167.64 195.58)
+		)
+		(stroke
+			(width 0)
+			(type default)
+		)
+	)
+	(wire
+		(pts
 			(xy 36.83 104.14) (xy 44.45 104.14)
 		)
@@
 	(wire
 		(pts
-			(xy 161.29 195.58) (xy 167.64 195.58)
-		)
-		(stroke
-			(width 0)
-			(type default)
-		)
-	)
-	(wire
-		(pts
 			(xy 176.53 95.25) (xy 175.26 95.25)
 		)
@@
 	(wire
 		(pts
-			(xy 158.75 200.66) (xy 161.29 200.66)
-		)
-		(stroke
-			(width 0)
-			(type default)
-		)
-	)
-	(wire
-		(pts
 			(xy 189.23 162.56) (xy 189.23 156.21)
 		)
@@
 	(wire
 		(pts
-			(xy 161.29 200.66) (xy 166.37 200.66)
-		)
-		(stroke
-			(width 0)
-			(type default)
-		)
-	)
-	(wire
-		(pts
 			(xy 350.52 212.09) (xy 350.52 224.79)
 		)
@@
 	(wire
 		(pts
+			(xy 161.29 200.66) (xy 166.37 200.66)
+		)
+		(stroke
+			(width 0)
+			(type default)
+		)
+	)
+	(wire
+		(pts
 			(xy 167.64 190.5) (xy 173.99 190.5)
 		)
@@
 	(wire
 		(pts
-			(xy 161.29 198.12) (xy 166.37 198.12)
-		)
-		(stroke
-			(width 0)
-			(type default)
-		)
-	)
-	(wire
-		(pts
 			(xy 54.61 242.57) (xy 54.61 245.11)
 		)
@@
 	(wire
 		(pts
-			(xy 158.75 198.12) (xy 161.29 198.12)
-		)
-		(stroke
-			(width 0)
-			(type default)
-		)
-	)
-	(wire
-		(pts
 			(xy 163.83 148.59) (xy 163.83 156.21)
 		)
@@
 		)
 		(instances
-			(project ""
+			(project "OPNhydro_r2"
 				(path "/a0000000-0000-4000-8000-000000002687"
 					(reference "M4")
