File: hardware/OPNhydro_r2/OPNhydro_r2.kicad_sch (KiCad schematic)
At the start: 164 parts, among them J2 MKDS, J3 BNC, J4 BNC, J5 BNC, M1 ESP32-C6-DEVKIT, M2 ATLAS_EZO_pH, M3 ATLAS_EZO_EC, M4 ATLAS_EZO_RTD, P1 MSTB_0.2", P10 ANKO_A200SX, P11 ANKO_A200SX, P12 ANKO_A200SX, P13 PB_1.25mm, P2 PHR_4, P3 MC_0.2", P4 DC40F-2460, P5 PHR_4, P6 MC_0.15", P7 XH_2.5mm, P8 XH_2.5mm, P9 XH_2.5mm, SW1 FLOAT, SW2 FLOAT, T1 AON6407, T2 BT3904, T3 IRLR2905, T4 BT3904, T5 AO3400A, U1 TPS62933, U2 AZ1117-3.3, U3 ADM3260, U4 ADM3260, U5 TMC2209, U6 TMC2209, U7 TMC2209

Commit message: update
Parts:
- removed H1: MSTBA_0.2", Coert-Vonk:TERM BLK HDR 2POS MSTBA 5.08mm, symbol Coert-Vonk:TERM BLK HDR 2POS MSTBA 5.08mm
- removed H3: MC_0.2", Coert-Vonk:TERM BLK HDR 2POS 5.08mm, symbol Coert-Vonk:TERM BLK HDR 2POS MC 5.08mm
- removed H5: MC_0.15", Coert-Vonk:TERM BLK HDR 2POS 3.81mm, symbol Coert-Vonk:TERM BLK HDR 2POS MC 3.81mm
- removed J2: MKDS, Coert-Vonk:TERM BLK 4POS SCREW 3.5mm, symbol Coert-Vonk:TERM BLK SCREW 4POS MKDS 3.5mm
- removed P1: MSTB_0.2", Coert-Vonk:TERM BLK PLG 2POS MSTB 5.08mm, symbol Coert-Vonk:TERM BLK PLG 2POS MSTB 5.08mm
- removed P3: MC_0.2", Coert-Vonk:TERM BLK PLUG 2POS 5.08mm, symbol Coert-Vonk:TERM BLK PLG 2POS MC 5.08mm
- removed P6: MC_0.15", Coert-Vonk:TERM BLOCK PLUG 2POS 3.81mm 1803578, symbol Coert-Vonk:TERM BLK PLG 2POS MC 3.81mm
- removed R24, R33: 110mΩ, Coert-Vonk:RES 0805 YAGEO, symbol Coert-Vonk:RES 110mΩ ±1% 1/8W 0805 Susumu
- added H1: MSTBA_0.2", Coert-Vonk:TERM BLK HDR 2POS MSTBA 5.08mm, symbol Coert-Vonk:TERM BLK HDR 2POS PC-MSTBA 0.2{dblquote}
- added H3, H5: MC_0.2", Coert-Vonk:TERM BLK HDR 2POS 5.08mm, symbol Coert-Vonk:TERM BLK HDR 2POS PC-MC 0.2{dblquote}
- added J1: SS-3.5mm, Coert-Vonk:TERM BLK 4POS SCREW 3.5mm, symbol Coert-Vonk:TERM BLK SCREW 4POS SS-MKDS 3.5mm
- added P1: MSTB_0.2", Coert-Vonk:TERM BLK PLG 2POS MSTB 5.08mm, symbol Coert-Vonk:TERM BLK PLG 2POS PC-MSTB 0.2{dblquote}
- added P3, P6: MC_0.2", Coert-Vonk:TERM BLK PLG 2POS PC-MC 0.2, symbol Coert-Vonk:TERM BLK PLG 2POS PC-MC 0.2{dblquote}
- added R24, R33: 110mΩ, Coert-Vonk:RES 0805 YAGEO, symbol Coert-Vonk:RES 110mΩ ±1% 1/4W 0805 Susumu
- C57: MFR (none) -> Murata; PN (none) -> GRM21BR61C106KE15L; SERIES (none) -> GRM
- FB1: MFR (none) -> Murata; PN (none) -> BLM31SN500SN1L; SERIES (none) -> BLM31
- T1: MFR (none) -> Alpha & Omega; PN (none) -> AON6407
Connections:
- net 24V: now also H3.1, H5.1
- net 3V3: now also J1.1 (Pin_1)
- net FLOAT_HIGH: now also J1.2 (Pin_2)
- net FLOAT_LOW: now also J1.3 (Pin_3)
- net GND: now also H1.2, J1.4 (Pin_4), R24.2, R33.2
- net at D3.A, T3.3 (D): now also H3.2
- net at D4.A, T5.3 (D): now also H5.2
- net at U5.23 (BRA): now also R24.1
- net at U5.27 (BRB): now also R33.1
- net at V1.24V: now also P6.1
- net at V1.GND: now also P6.2
- net at P4.24V: now also P3.1
- net at P4.GND: now also P3.2
- net at FB1.1: now also H1.1
- net at DC1.24V: now also P1.1
- net at DC1.GND: now also P1.2

Commit message: update
Parts:
- removed C4: 1000μF, Coert-Vonk:CAP ALUM 1000μF ±20 50V Panasonic, symbol Coert-Vonk:CAP ALUM-ELEC 1000μF ±20% 50V Panasonic
- added C4: 1000μF, Coert-Vonk:CAP ALUM-ELEC 1000μF ±20 50V TDK, symbol Coert-Vonk:CAP ALUM-ELEC 1000μF ±20% 50V TDK
- C1: footprint Coert-Vonk:CAP ALUM 100μF ±20 25V -> Coert-Vonk:CAP ALUM 100μF ±20 10V Kemet; symbol Coert-Vonk:CAP ALUM-ELEC 100μF ±20% 25V Panasonic -> Coert-Vonk:CAP ALUM-ELEC 100μF ±20% 10V Kemet; DKPN 10-EEE-FN1E101UPCT-ND -> 399-A750BK107M1AAAE024-ND; MFR (none) -> Kemet; MOUNT (none) -> Radial; PN (none) -> A750BK107M1AAAE024; SERIES (none) -> A750
- C10, C16, C18, C2, C20, C22, C26, C28, C3, C32, C34, C35, C39, C40, C44, C45, C46, C47, C48, C49, C50, C51, C52, C56, C58, C6, C61, C9: footprint Coert-Vonk:CAP X7R 100nF ±10 50V 0402 Murata -> Coert-Vonk:CAP X7R 100nF ±10 50V 0603 Murata; symbol Coert-Vonk:CAP X7R 100nF ±10% 50V 0402 Murata -> Coert-Vonk:CAP X7R 100nF ±10% 100V 0603 Murata; DKPN 490-10700-1-ND -> 490-3285-1-ND; MFR (none) -> Murata; MOUNT (none) -> 0603; PN (none) -> GRM188R72A104KA35D; SERIES (none) -> GRM
- C11: SERIES (none) -> GRM
- C12: footprint Coert-Vonk:CAP ALUM 220μF ±20 50V Panasonic -> Coert-Vonk:CAP ALUM 220μF ±20 50V Kemet; symbol Coert-Vonk:CAP ALUM-ELEC 220μF ±20% 50V Panasonic -> Coert-Vonk:CAP ALUM-ELEC 220μF ±20% 50V Kemet; DKPN 10-ECA-1HM221BCT-ND -> 399-6123-ND; MFR Panasonic -> Kemet; MOUNT (none) -> Radial; PN ECA-1HM221B -> ESY227M050AH2AA; SERIES (none) -> ESY
- C13, C14, C17, C19, C31, C33, C59: MFR (none) -> Murata; PN (none) -> GRM21BR61C106KE15L; SERIES (none) -> GRM
- C21: footprint Coert-Vonk:CAP X7R 10nF ±10 16V 0402 Murata -> Coert-Vonk:CAP X7R 10nF ±10 100V 0603 Murata; symbol Coert-Vonk:CAP X7R 10nF ±10% 16V 0402 Murata -> Coert-Vonk:CAP X7R 10nF ±10% 100V 0603 Murata; DKPN 490-1313-1-ND -> 490-GRM188R72A103KA01JCT-ND; MFR (none) -> Murata; PN GRM155R71C103KA01D -> GRM188R72A103KA01J; SERIES (none) -> GRM
- C23, C27, C29: footprint Coert-Vonk:CAP X7R 10nF ±10 16V 0402 Murata -> Coert-Vonk:CAP X7R 10nF ±10 100V 0603 Murata; symbol Coert-Vonk:CAP X7R 10nF ±10% 16V 0402 Murata -> Coert-Vonk:CAP X7R 10nF ±10% 100V 0603 Murata; DKPN 490-1313-1-ND -> 490-GRM188R72A103KA01JCT-ND; MFR (none) -> Murata; PN (none) -> GRM188R72A103KA01J; SERIES (none) -> GRM
- C24: MOUNT (none) -> SMD; SERIES (none) -> OS-CON, SVPK
- C25: MFR (none) -> Murata; PN (none) -> GRM31CR71A226KE15L
- C30: footprint Coert-Vonk:CAP ALUM-ELEC 47μF ±20 50V Panasonic -> Coert-Vonk:CAP ALUM-ELEC 47μF ±20 50V Kemet; symbol Coert-Vonk:CAP ALUM-ELEC 47μF ±20% 50V Panasonic -> Coert-Vonk:CAP ALUM-ELEC 47μF ±20% 50V Kemet; DKPN 10-ECA-1HM470ICT-ND -> 399-ESY476M050AE3AA-ND; MFR Panasonic -> KEMET; MOUNT (none) -> Radial; PN ECA-1HM470I -> ESY476M050AE3AA; SERIES (none) -> ESY
- C36, C37, C38: MFR (none) -> Murata; PN (none) -> GRM188R71A225KE15J; SERIES (none) -> GRM
- C41, C42, C43: MFR (none) -> Murata; MOUNT (none) -> 0603; PN (none) -> GRM188R72A223KAC4D; SERIES (none) -> GRM
- C53, C54, C55: footprint Coert-Vonk:CAP ALUM 220μF ±20 50V Panasonic -> Coert-Vonk:CAP ALUM 220μF ±20 50V Kemet; symbol Coert-Vonk:CAP ALUM-ELEC 220μF ±20% 50V Panasonic -> Coert-Vonk:CAP ALUM-ELEC 220μF ±20% 50V Kemet; DKPN 10-ECA-1HM221BCT-ND -> 399-6123-ND; MFR (none) -> Kemet; MOUNT (none) -> Radial; PN (none) -> ESY227M050AH2AA; SERIES (none) -> ESY
- C7: footprint Coert-Vonk:CAP X7R 33nF ±10 50V 0805 Kemet -> Coert-Vonk:CAP X7R 33nF ±10 50V 0603 Kemet; symbol Coert-Vonk:CAP X7R 33nF ±10% 50V 0805 Kemet -> Coert-Vonk:CAP X7R 33nF ±10% 50V 0603 Kemet; DKPN 490-GRM155R71H333KE14JCT-ND -> 399-C0603C333K5RACTUCT-ND; MFR Murata -> Kemet; MOUNT (none) -> 0603; PN GRM155R71H333KE14J -> C0603C333K5RACTU; SERIES (none) -> SMD Comm X7R
- C8: footprint Coert-Vonk:CAP X7R 100nF ±10 50V 0402 Murata -> Coert-Vonk:CAP X7R 100nF ±10 50V 0603 Murata; symbol Coert-Vonk:CAP X7R 100nF ±10% 50V 0402 Murata -> Coert-Vonk:CAP X7R 100nF ±10% 100V 0603 Murata; DKPN 490-10700-1-ND -> 490-3285-1-ND; MOUNT (none) -> 0603; PN GRM155R71H104KE14D -> GRM188R72A104KA35D; SERIES (none) -> GRM
- D1: MFR (none) -> Diodes; PN (none) -> SMBJ28A-13-F; SERIES (none) -> SMBJ
- D2: MFR (none) -> Diodes; PN (none) -> BZT52C12S-7-F
- D3, D4: MFR (none) -> Onsemi; PN (none) -> SS34
- F1: MFR (none) -> Littelfuse; PN (none) -> 0451007.MRL; SERIES (none) -> NANO 451
- FB2: footprint (none) -> Coert-Vonk:FERRITE BEAD 20mΩ 60Ω 0603 TDK; MPN (none) -> MPZ1608S600ATDH5
- FB3, FB4, FB5: footprint (none) -> Coert-Vonk:FERRITE BEAD 20mΩ 60Ω 0603 TDK
- H6, H7, H8: MFR (none) -> JST; PN (none) -> S4B-XH-A
- J1: SERIES (none) -> TB0011-350
- J3, J4, J5: MFR (none) -> TE Connectivity
- L1: MFR (none) -> Bourns; PN (none) -> SDR1307-100ML
- M1: MFR (none) -> Espressif Systems; PN (none) -> ESP32-C6-DEVKITC-1-N8; SERIES (none) -> ESP32-C
- M2: MFR (none) -> Atlas Scientific; PN (none) -> EZO-PH
- P2, P5: MFR (none) -> JST; PN (none) -> PHR-4; SERIES (none) -> PH
- P7, P8, P9: footprint Coert-Vonk:TERM BLK PLG 4POS XH 2.5mm -> Coert-Vonk:TERM BLK PLG 4POS JST-XH 2.5mm; MFR (none) -> JST; PN (none) -> XHP-4
- R1, R14, R15, R16, R2: MFR (none) -> Yageo; PN (none) -> RC0805FR-072K2L; SERIES (none) -> RC_L
- R11: MFR (none) -> Yageo; PN (none) -> RC0805FR-0752K3L
- R12, R19, R20, R23, R3, R6: MFR (none) -> Yageo; PN (none) -> RC0805FR-0710KL; SERIES (none) -> RC_L
- R13: PN (none) -> RC0805FR-072K2L
- R17, R18: MFR (none) -> Yageo; PN (none) -> RC0805FR-0716K9L; SERIES (none) -> RC_L
- R21: DKPN 100 Ohms ±1% 0.125W, 1/8W Chip Resistor 0805 (2012 Metric) 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 -> 311-100CRCT-ND; MGR (none) -> Yageo; PN (none) -> RC0805FR-07100RL; SERIES (none) -> RC_L
- R22, R9: MFR (none) -> Yageo; PN (none) -> RC0805FR-074K7L; SERIES (none) -> RC_L
- R24, R33: MFR (none) -> Susumu; PN (none) -> RL1220S-R11-F; SERIES (none) -> RL
- R27, R29, R31: MFR (none) -> Yageo; PN (none) -> RC0805FR-1014KL; SERIES (none) -> RC_L
- R4: MFR (none) -> Yageo; PN (none) -> RC0805FR-1333KL; SERIES (none) -> RC_L
- R5: MFR (none) -> Yageo; PN (none) -> RC0805FR-071KL; SERIES (none) -> RC_L
- R8: DKPN (none) -> 311-100CRCT-ND; MGR (none) -> Yageo; PN (none) -> RC0805FR-07100RL; SERIES (none) -> RC_L
- T3: MFR (none) -> Infineon; PN (none) -> IRLR2905TRPBF; SERIES (none) -> HEXFET
- T5: MFR (none) -> Alpha & Omega; PN (none) -> AO3400A
- U4: MFR (none) -> Analog Devices; PN (none) -> ADM3260ARSZ; SERIES (none) -> IsoPower
- U5, U6, U7: MFR (none) -> Analog Devices; PN (none) -> TMC2209-LA-T; SERIES (none) -> stallGuard
Connections:
- net 24V: now also C4.1
- net GND: now also C4.2

Commit message: update
Parts:
- added FID1, FID2, FID3: Fiducial, symbol Mechanical:Fiducial
- added MH1, MH2, MH3, MH4: M3, MountingHole:MountingHole_3.2mm_M3_Pad_Via, symbol Mechanical:MountingHole_Pad
- C1: value 100μF -> 100μ; DIGIKEY (none) -> 399-A750BK107M1AAAE024-ND; LCSC (none) -> C1020041
- C10, C16, C18, C2, C20, C22, C26, C28, C3, C32, C34, C35, C39, C40, C44, C45, C46, C47, C48, C49, C50, C51, C52, C56, C58, C61, C8, C9: value 100nF -> 100n; LCSCPN (none) -> C77058
- C11, C13, C14, C15, C17, C19, C31, C33, C57, C59: value 10μF -> 10μ; symbol Coert-Vonk:CAP X5R 10μF ±10% 16V 0805 Murata GRM -> Coert-Vonk:CAP X5R 10μF ±10% 16V 0805 Murata; DIGIKEY (none) -> 490-3886-1-ND; LCSC (none) -> C77075; PKG (none) -> 0805
- C12: value 220μF -> 220μ; DIGIKEY (none) -> 399-6123-ND; LCSC (none) -> C5113406; MFR Kemet -> KEMET
- C21, C23, C27, C29: value 10nF -> 10n; DIGIKEY (none) -> 490-GRM188R72A103KA01JCT-ND; LCSC (none) -> C2187930; PKG (none) -> 0603
- C24: value 220μF -> 220μ; DIGIKEY (none) -> P124158CT-ND; LCSC (none) -> C542293
- C25: value 22μF -> 22μ; symbol Coert-Vonk:CAP X7R 22μF ±10% 10V 1206 Murata GRM -> Coert-Vonk:CAP X7R 22μF ±10% 10V 1206 Murata; LCSC (none) -> C91604; PKG (none) -> 1206; SERIES (none) -> GRM
- C30: value 47μF -> 47μ; DIGIKEY (none) -> 399-ESY476M050AE3AA-ND; LCSC (none) -> C1019527
- C36, C37, C38: value 2.2μF -> 2μ2; LCSC (none) -> C2167658; MOUNT (none) -> 0603
- C4: value 1000μF -> 1000μ; DIGIKEY (none) -> B41866D6108M000; LCSCPN (none) -> C1650604
- C5: value 10μF -> 10μ; symbol Coert-Vonk:CAP X7R 10μF ±10% 50V 1206 Murata GRT -> Coert-Vonk:CAP X7R 10μF ±10% 50V 1206 Murata; DIGIKEY (none) -> 490-12456-1-ND; LCSC (none) -> C417124; LCSCPN (none) -> C417124; PKG (none) -> 1206; SERIES (none) -> GRT
- C53, C54, C55: value 220μF/50V -> 220μ; DIGIKEY (none) -> 399-6123-ND; LCSC (none) -> C5113406; MFR Kemet -> KEMET
- C6: value 100nF -> 100n; DIGIKEY (none) -> 490-3285-1-ND; LCSC (none) -> C77058; LCSCPN (none) -> C77058
- C7: value 33nF -> 33n; DIGIKEY (none) -> 399-C0603C333K5RACTUCT-ND; LCSC (none) -> C2169037; MFR Kemet -> KEMET
- D1: DIGIKEY (none) -> SMBJ28A-FDICT-ND; LCSC (none) -> C91924; MOUNT (none) -> DO-214AA
- D3, D4: DIGIKEY (none) -> SS34FSCT-ND; LCSC (none) -> C154551; PKG (none) -> DO-214AB, SMC
- DC1: DIGIKEY (none) -> 1866-3321-ND; LCSC (none) -> C95193; MFR (none) -> MEAN WELL USA Inc.; PN (none) -> LRS-150-24; SERIES (none) -> LRS-150 (150W)
- FB1: value 50Ω@100Mhz/12A -> 50Ω@100Mhz; DIGIKEY (none) -> 490-13269-1-ND; LCSC (none) -> C710524; MOUNT (none) -> 1206
- FB2: DIGIKEY (none) -> 445-MPZ1608S600ATDH5CT-ND; LCSC (none) -> C307775; PKG (none) -> 0603
- FB3, FB4, FB5: DIGIKEY (none) -> 445-MPZ1608S600ATDH5CT-ND; LCSC (none) -> C307775; PKG (none) -> 0603; SERIES (none) -> MPZ
- H1: DIGIKEY (none) -> 277-1106-ND; LCSC (none) -> C90074
- H9: DIGIKEY (none) -> WM7624CT-ND; LCSC (none) -> C17393620; PN (none) -> 0532610671; SERIES (none) -> PicoBlade 53261
- J3, J4, J5: DIGIKEY (none) -> A32259-ND; PN (none) -> 5227161-6; SLSC (none) -> C5166169
- L1: value 10µH -> 10µ; DIGIKEY (none) -> SDR1307-100MLCT-ND; LCSC (none) -> C49672242; PKG (none) -> Nonstandard SMD
- M1: DIGIKEY (none) -> 1965-ESP32-C6-DEVKITC-1-N8-ND; LCSC (none) -> C20554022; PKG (none) -> Mezzanine
- M2: DIGIKEY (none) -> 5016-EZO-PH-ND; SERIES (none) -> EZO
- M3: DIGIKEY (none) -> 5016-EZO-EC-ND; MFR (none) -> Atlas Scientific; PN (none) -> EZO-EC; SERIES (none) -> EZO
- M4: DIGIKEY (none) -> 5016-EZO-RTD-ND; MFR (none) -> Atlas Scientific; PN (none) -> EZO-RTD; SERIES (none) -> EZO
- P1: DIGIKEY (none) -> 277-1011-ND; LCSC (none) -> C90073
- P13: DIGIKEY (none) -> WM1724-ND; LCSC (none) -> C385105; PN (none) -> 0510210600; SERIES (none) -> PicoBlade 51021
- PR1: MFR (none) -> Benewake; PN (none) -> TF-Luna; SERIES (none) -> TF
- PR3: MFR (none) -> Bluelab; PN (none) -> PROBPH
- PR4: MFR (none) -> Bluelab; PN (none) -> PROBPCEC
- PR5: DIGIKEY (none) -> 5016-PT-1000-ND; MFR (none) -> Atlas Scientific; PN (none) -> PT-1000
- R1, R13, R14, R15, R16, R2: DIGIKEY (none) -> 311-2.20KCRCT-ND; LCSC (none) -> C114561; PKG (none) -> 0805
- R10, R12, R19, R20, R23, R3, R6: DIGIKEY (none) -> 311-10.0KCRCT-ND; LCSC (none) -> C84376; PKG (none) -> 0805
- R11: DIGIKEY (none) -> 311-52.3KCRCT-ND; LCSC (none) -> C273887; PKG (none) -> 0805; SERIES (none) -> RC_L
- R17, R18: DIGIKEY (none) -> 311-16.9KCRCT-ND; LCSC (none) -> C273834; PKG (none) -> 0805
- R21, R8: DIGIKEY (none) -> 311-100CRCT-ND; LCSC (none) -> C105577; PKG (none) -> 0805
- R22, R9: DIGIKEY (none) -> 311-4.70KCRCT-ND; LCSC (none) -> C60816; PKG (none) -> 0805
- R24, R33: LCSC (none) -> C2074624; PKG (none) -> 0805
- R27, R29, R31: DIGIKEY (none) -> 13-RC0805FR-1014KLCT-ND; LCSC (none) -> C4347440; PKG (none) -> 0805
- R28, R30, R32: DIGIKEY (none) -> 311-10.7KCRCT-ND; LCSC (none) -> C273918; MFR (none) -> Yageo; PKG (none) -> 0805; PN (none) -> RC0805FR-0710K7L; SERIES (none) -> RC_L
- R4: DIGIKEY (none) -> 13-RC0805FR-1333KLCT-ND; LCSC (none) -> C4245127; MOUNT (none) -> 0805
- R5: DIGIKEY (none) -> 311-1.00KCRCT-ND; LCSC (none) -> C95781; PKG (none) -> 0805
- R7: DIGIKEY (none) -> 311-21.0KCRCT-ND; LCSC (none) -> C137569; PKG (none) -> 0805; SERIES (none) -> RC_L
- T1: DIGIKEY (none) -> 785-1421-1-ND; LCSC (none) -> C13899; MOUNT (none) -> 8-DFN (5x6)
- T2: O (none) -> Onsemi; PKG (none) -> SOT-23-3
- T4: MFR (none) -> Onsemi; O (none) -> Onsemi; PKG (none) -> SOT-23-3; PN (none) -> MMBT3904LT1G
- T5: DIGIKEY (none) -> 785-1000-1-ND; LCSC (none) -> C20917; PKG (none) -> SOT-23-3
- U1: LCSC (none) -> C3200405; PKG (none) -> SOT-583
- U2: DIGIKEY (none) -> AZ1117IH-3.3TRG1DICT-ND; LCSC (none) -> C108495; PKG (none) -> SOT-223-3; SERIES (none) -> AZ1117I
- U3, U4: DIGIKEY (none) -> 505-ADM3260ARSZ-ND; LCSC (none) -> C208558; PKG (none) -> 20-SSOP
- U5, U6, U7: LCSC (none) -> C2150710; PKG (none) -> 28-VFQFN Exposed Pad
Connections:
- net GND: now also MH1.1, MH2.1, MH3.1, MH4.1
- net B_{NB}-: now reaches H8.4, U7.1 (OB2)
- net VREF_{NB}: now reaches R31.1, R32.2, U7.17 (VREF)
- net A_{NB}-: now reaches H8.2, U7.21 (OA2)
- net BRA_{NB}: now reaches R34.1, U7.23 (BRA)
- net A_{NB}+: now reaches H8.1, U7.24 (OA1)
- net B_{NB}+: now reaches H8.3, U7.26 (OB1)
- net BRB_{NB}: now reaches R35.1, U7.27 (BRB)
- net CP0_{NB}: now reaches C43.1, U7.4 (CPO)
- net CP1_{NB}: now reaches C43.2, U7.5 (CPI)
- net VCP_{NB}: now reaches C46.1, U7.6 (VCP)
- net 5V_{NB}: now reaches C37.2, R31.2, U7.8 (5VOUT)
- net GND_{EC}: now reaches FB5.1, M3.1 (GND)
- net SCL_{EC}: now reaches M3.2 (TX/SCL), R16.1, U4.19 (SCL_{1})
- net SDA_{EC}: now reaches M3.3 (RX/SDA), R14.1, U4.18 (SDA_{1})
- net PGND_{EC}: now reaches J4.G (GND), M3.4 (PGND)
- net PRB_{EC}: now reaches J4.S, M3.5 (PRB)
- net B_{PUMP}: now reaches R9.2, T2.1 (B)
- net VREF_{pH}: now reaches R27.1, R28.2, U5.17 (VREF)
- net 5V_{pH}: now reaches C38.2, R27.2, U5.8 (5VOUT)
- net D_{PUMP}: now reaches D3.A, H3.2, T3.3 (D)
- net A_{pH}+: now reaches H6.1, U5.24 (OA1)
- net A_{pH}: now reaches H6.2, U5.21 (OA2)
- net B_{pH}+: now reaches H6.3, U5.26 (OB1)
- net B_{pH}-: now reaches H6.4, U5.1 (OB2)
- net +5V_{BK}: now reaches C8.2, L1.1, U1.5 (SW)
- net GNDISO_{EC}: now reaches C17.1, C18.2, C22.1, C23.2, FB5.2, R20.2, U4.11 (GND_{ISO}), U4.14 (GND_{ISO}), U4.16 (GND_{ISO}), U4.20 (GND_{ISO})
- net VISO_{EC}: now reaches C17.2, C22.2, FB4.2, U4.12 (V_{ISO})
- net VSEL_{EC}: now reaches R18.1, R20.1, U4.13 (VSEL)
- net SCL_{pH}: now reaches M2.2 (TX/SCL), R15.1, U3.19 (SCL_{1})
- net G_{ATO}: now reaches R21.2, R23.2, T4.3 (C), T5.1 (G)
- net D_{ATO}: now reaches D4.A, H5.2, T5.3 (D)
- net BRA_{pH}: now reaches R24.1, U5.23 (BRA)
- net BRB_{pH}: now reaches R33.1, U5.27 (BRB)
- net CP0_{pH}: now reaches C41.1, U5.4 (CPO)
- net CP1_{pH}: now reaches C41.2, U5.5 (CPI)
- net VCP_{pH}: now reaches C44.1, U5.6 (VCP)
- net VISO_{pH}: now reaches C15.2, C20.2, FB2.2, U3.12 (V_{ISO})
- net G_{PUMP}: now reaches R10.1, R8.2, T2.3 (C), T3.1 (G)
- net +24V_{FB}: now reaches F1.1, FB1.2
- net +24V_{F}: now reaches D1.1 (C), F1.2, R4.2, T1.2 (S)
- net GND_{pH}: now reaches FB3.1, M2.1 (GND)
- net SDA_{pH}: now reaches M2.3 (RX/SDA), R13.1, U3.18 (SDA_{1})
- net PGND_{pH}: now reaches J3.G (GND), M2.4 (PGND)
- net PRB_{pH}: now reaches J3.S, M2.5 (PRB)
- net BRA_{NA}: now reaches R25.1, U6.23 (BRA)
- net A_{NA}+: now reaches H7.1, U6.24 (OA1)
- net A_{NA}-: now reaches H7.2, U6.21 (OA2)
- net B_{NA}+: now reaches H7.3, U6.26 (OB1)
- net B_{NA}-: now reaches H7.4, U6.1 (OB2)
- net GNDISO_{pH}: now reaches C15.1, C16.2, C20.1, C21.2, FB3.2, R19.2, U3.11 (GND_{ISO}), U3.14 (GND_{ISO}), U3.16 (GND_{ISO}), U3.20 (GND_{ISO})
- net VREF_{NA}: now reaches R29.1, R30.2, U6.17 (VREF)
- net BRB_{NA}: now reaches R26.1, U6.27 (BRB)
- net CP0_{NA}: now reaches C42.1, U6.4 (CPO)
- net CP1_{NA}: now reaches C42.2, U6.5 (CPI)
- net VCP_{NA}: now reaches C45.1, U6.6 (VCP)
- net 5V_{NA}: now reaches C36.2, R29.2, U6.8 (5VOUT)
- net G_{RPP}: now reaches D2.1 (K), R4.1, T1.1 (G)
- net BST_{BK}: now reaches C8.1, U1.6 (BST)
- net B_{ATO}: now reaches R22.2, T4.1 (B)
- net SS_{BK}: now reaches C7.2, U1.7 (SS)
- net VSEL_{pH}: now reaches R17.1, R19.1, U3.13 (VSEL)
- net PGND_{T}: now reaches J5.G (GND), M4.4 (PGND)
- net PRB_{T}: now reaches J5.S, M4.5 (PRB)
- net RT_{BK}: now reaches R7.2, U1.1 (RT)
- net 0V8 renamed 0V8_{BK}
- net 24V renamed +24V
- net 3V3 renamed +3V3
- net 5V renamed +5V
- net V_{ISO,EC} renamed V_{EC}
- net V_{ISO,pH} renamed V_{pH}
Other:
- note removed: "Noise mitigation"
- note removed: "bulk for WiFi Tx"
- note removed: "bulk for simultaneous motors"
- note removed: "f_{SW}=1MHz"
- note removed: "t_{ss}=5ms"
- moved on the sheet: C8, L1, R21, R22, R24, R33, T2

Commit message: update
Parts:
- removed R25, R26, R34, R35: 110mΩ, Coert-Vonk:RES 0805 YAGEO, symbol Coert-Vonk:RES 110mΩ ±1% 1/8W 0805 Susumu
- added R30, R31, R32, R33: 110mΩ, Coert-Vonk:RES 0805 YAGEO, symbol Coert-Vonk:RES 110mΩ ±1% 1/4W 0805 Susumu
- C1: DKPN 399-A750BK107M1AAAE024-ND -> (none); MFR Kemet -> (none); MOUNT Radial -> (none); PKG (none) -> Radial
- C10: renamed from C7; DKPN 399-C0603C333K5RACTUCT-ND -> (none); MFR KEMET -> (none); MOUNT 0603 -> (none); PKG (none) -> 0603
- C11: renamed from C61; DIGIKEY (none) -> 490-3285-1-ND; DKPN 490-3285-1-ND -> (none); LCSC (none) -> C77058; LCSCPN C77058 -> (none); MFR Murata -> (none); MOUNT 0603 -> (none); PKG (none) -> 0603
- C12: renamed from C8; DIGIKEY (none) -> 490-3285-1-ND; DKPN 490-3285-1-ND -> (none); LCSC (none) -> C77058; LCSCPN C77058 -> (none); MFR Murata -> (none); MOUNT 0603 -> (none); PKG (none) -> 0603
- C13: renamed from C10; DIGIKEY (none) -> 490-3285-1-ND; DKPN 490-3285-1-ND -> (none); LCSC (none) -> C77058; LCSCPN C77058 -> (none); MFR Murata -> (none); MOUNT 0603 -> (none); PKG (none) -> 0603
- C14: renamed from C13; DKPN 490-3886-1-ND -> (none); MFR Murata -> (none)
- C15: renamed from C11; DKPN 490-3886-1-ND -> (none); MFR Murata -> (none)
- C16: renamed from C14; DKPN 490-3886-1-ND -> (none); MFR Murata -> (none)
- C17: renamed from C15; DKPN 490-3886-1-ND -> (none); MFR Murata -> (none)
- C18: renamed from C16; DIGIKEY (none) -> 490-3285-1-ND; DKPN 490-3285-1-ND -> (none); LCSC (none) -> C77058; LCSCPN C77058 -> (none); MFR Murata -> (none); MOUNT 0603 -> (none); PKG (none) -> 0603
- C19: renamed from C17; DKPN 490-3886-1-ND -> (none); MFR Murata -> (none)
- C2: renamed from C12; DKPN 399-6123-ND -> (none); MFR KEMET -> (none); MOUNT Radial -> (none); PKG (none) -> Radial; Series M-A -> (none)
- C20: renamed from C18; DIGIKEY (none) -> 490-3285-1-ND; DKPN 490-3285-1-ND -> (none); LCSC (none) -> C77058; LCSCPN C77058 -> (none); MFR Murata -> (none); MOUNT 0603 -> (none); PKG (none) -> 0603
- C21: renamed from C19; DKPN 490-3886-1-ND -> (none); MFR Murata -> (none)
- C22: renamed from C20; DIGIKEY (none) -> 490-3285-1-ND; DKPN 490-3285-1-ND -> (none); LCSC (none) -> C77058; LCSCPN C77058 -> (none); MFR Murata -> (none); MOUNT 0603 -> (none); PKG (none) -> 0603
- C23: renamed from C21; DKPN 490-GRM188R72A103KA01JCT-ND -> (none); MFR Murata -> (none)
- C24: renamed from C22; DIGIKEY (none) -> 490-3285-1-ND; DKPN 490-3285-1-ND -> (none); LCSC (none) -> C77058; LCSCPN C77058 -> (none); MFR Murata -> (none); MOUNT 0603 -> (none); PKG (none) -> 0603
- C25: renamed from C23; DKPN 490-GRM188R72A103KA01JCT-ND -> (none); MFR Murata -> (none)
- C26: renamed from C24; DKPN P124158CT-ND -> (none); MFR Panasonic -> (none); MOUNT SMD -> (none); PKG (none) -> SMD
- C27: renamed from C25; DKPN 490-5309-1-ND -> (none); MFR Murata -> (none)
- C28: renamed from C56; DIGIKEY (none) -> 490-3285-1-ND; DKPN 490-3285-1-ND -> (none); LCSC (none) -> C77058; LCSCPN C77058 -> (none); MFR Murata -> (none); MOUNT 0603 -> (none); PKG (none) -> 0603
- C29: renamed from C58; DIGIKEY (none) -> 490-3285-1-ND; DKPN 490-3285-1-ND -> (none); LCSC (none) -> C77058; LCSCPN C77058 -> (none); MFR Murata -> (none); MOUNT 0603 -> (none); PKG (none) -> 0603
- C3: renamed from C9; DIGIKEY (none) -> 490-3285-1-ND; DKPN 490-3285-1-ND -> (none); LCSC (none) -> C77058; LCSCPN C77058 -> (none); MFR Murata -> (none); MOUNT 0603 -> (none); PKG (none) -> 0603
- C30: renamed from C57; DKPN 490-3886-1-ND -> (none); MFR Murata -> (none)
- C31: renamed from C59; DKPN 490-3886-1-ND -> (none); MFR Murata -> (none)
- C32: renamed from C26; DIGIKEY (none) -> 490-3285-1-ND; DKPN 490-3285-1-ND -> (none); LCSC (none) -> C77058; LCSCPN C77058 -> (none); MFR Murata -> (none); MOUNT 0603 -> (none); PKG (none) -> 0603
- C33: renamed from C27; DKPN 490-GRM188R72A103KA01JCT-ND -> (none); MFR Murata -> (none)
- C34: renamed from C28; DIGIKEY (none) -> 490-3285-1-ND; DKPN 490-3285-1-ND -> (none); LCSC (none) -> C77058; LCSCPN C77058 -> (none); MFR Murata -> (none); MOUNT 0603 -> (none); PKG (none) -> 0603
- C35: renamed from C29; DKPN 490-GRM188R72A103KA01JCT-ND -> (none); MFR Murata -> (none)
- C36: renamed from C31; DKPN 490-3886-1-ND -> (none); MFR Murata -> (none)
- C37: renamed from C32; DIGIKEY (none) -> 490-3285-1-ND; DKPN 490-3285-1-ND -> (none); LCSC (none) -> C77058; LCSCPN C77058 -> (none); MFR Murata -> (none); MOUNT 0603 -> (none); PKG (none) -> 0603
- C38: renamed from C33; DKPN 490-3886-1-ND -> (none); MFR Murata -> (none)
- C39: renamed from C34; DIGIKEY (none) -> 490-3285-1-ND; DKPN 490-3285-1-ND -> (none); LCSC (none) -> C77058; LCSCPN C77058 -> (none); MFR Murata -> (none); MOUNT 0603 -> (none); PKG (none) -> 0603
- C4: renamed from C2; DIGIKEY (none) -> 490-3285-1-ND; DKPN 490-3285-1-ND -> (none); LCSC (none) -> C77058; LCSCPN C77058 -> (none); MFR Murata -> (none); MOUNT 0603 -> (none); PKG (none) -> 0603
- C40: renamed from C38; DIGIKEY (none) -> 490-6418-1-ND; DKPN 490-6418-1-ND -> (none); MFR Murata -> (none); MOUNT 0603 -> (none); PKG (none) -> 0603
- C41: renamed from C36; DIGIKEY (none) -> 490-6418-1-ND; DKPN 490-6418-1-ND -> (none); MFR Murata -> (none); MOUNT 0603 -> (none); PKG (none) -> 0603
- C42: renamed from C37; DIGIKEY (none) -> 490-6418-1-ND; DKPN 490-6418-1-ND -> (none); MFR Murata -> (none); MOUNT 0603 -> (none); PKG (none) -> 0603
- C43: renamed from C35; DIGIKEY (none) -> 490-3285-1-ND; DKPN 490-3285-1-ND -> (none); LCSC (none) -> C77058; LCSCPN C77058 -> (none); MFR Murata -> (none); MOUNT 0603 -> (none); PKG (none) -> 0603
- C44: renamed from C39; DIGIKEY (none) -> 490-3285-1-ND; DKPN 490-3285-1-ND -> (none); LCSC (none) -> C77058; LCSCPN C77058 -> (none); MFR Murata -> (none); MOUNT 0603 -> (none); PKG (none) -> 0603
- C45: renamed from C40; DIGIKEY (none) -> 490-3285-1-ND; DKPN 490-3285-1-ND -> (none); LCSC (none) -> C77058; LCSCPN C77058 -> (none); MFR Murata -> (none); MOUNT 0603 -> (none); PKG (none) -> 0603
- C46: renamed from C41; value 22nF -> 22n; DIGIKEY (none) -> 490-3284-1-ND; DKPN 490-3284-1-ND -> (none); LCSC (none) -> C426087; MFR Murata -> (none); MOUNT 0603 -> (none); PKG (none) -> 0603
- C47: renamed from C42; value 22nF -> 22n; DIGIKEY (none) -> 490-3284-1-ND; DKPN 490-3284-1-ND -> (none); LCSC (none) -> C426087; MFR Murata -> (none); MOUNT 0603 -> (none); PKG (none) -> 0603
- C48: renamed from C43; value 22nF -> 22n; DIGIKEY (none) -> 490-3284-1-ND; DKPN 490-3284-1-ND -> (none); LCSC (none) -> C426087; MFR Murata -> (none); MOUNT 0603 -> (none); PKG (none) -> 0603
- C49: renamed from C44; DIGIKEY (none) -> 490-3285-1-ND; DKPN 490-3285-1-ND -> (none); LCSC (none) -> C77058; LCSCPN C77058 -> (none); MFR Murata -> (none); MOUNT 0603 -> (none); PKG (none) -> 0603
- C5: renamed from C3; DIGIKEY (none) -> 490-3285-1-ND; DKPN 490-3285-1-ND -> (none); LCSC (none) -> C77058; LCSCPN C77058 -> (none); MFR Murata -> (none); MOUNT 0603 -> (none); PKG (none) -> 0603
- C50: renamed from C45; DIGIKEY (none) -> 490-3285-1-ND; DKPN 490-3285-1-ND -> (none); LCSC (none) -> C77058; LCSCPN C77058 -> (none); MFR Murata -> (none); MOUNT 0603 -> (none); PKG (none) -> 0603
- C51: renamed from C46; DIGIKEY (none) -> 490-3285-1-ND; DKPN 490-3285-1-ND -> (none); LCSC (none) -> C77058; LCSCPN C77058 -> (none); MFR Murata -> (none); MOUNT 0603 -> (none); PKG (none) -> 0603
- C52: renamed from C47; DIGIKEY (none) -> 490-3285-1-ND; DKPN 490-3285-1-ND -> (none); LCSC (none) -> C77058; LCSCPN C77058 -> (none); MFR Murata -> (none); MOUNT 0603 -> (none); PKG (none) -> 0603
- C53: renamed from C48; DIGIKEY (none) -> 490-3285-1-ND; DKPN 490-3285-1-ND -> (none); LCSC (none) -> C77058; LCSCPN C77058 -> (none); MFR Murata -> (none); MOUNT 0603 -> (none); PKG (none) -> 0603
- C54: renamed from C49; DIGIKEY (none) -> 490-3285-1-ND; DKPN 490-3285-1-ND -> (none); LCSC (none) -> C77058; LCSCPN C77058 -> (none); MFR Murata -> (none); MOUNT 0603 -> (none); PKG (none) -> 0603
- C55: renamed from C50; DIGIKEY (none) -> 490-3285-1-ND; DKPN 490-3285-1-ND -> (none); LCSC (none) -> C77058; LCSCPN C77058 -> (none); MFR Murata -> (none); MOUNT 0603 -> (none); PKG (none) -> 0603
- C56: renamed from C51; DIGIKEY (none) -> 490-3285-1-ND; DKPN 490-3285-1-ND -> (none); LCSC (none) -> C77058; LCSCPN C77058 -> (none); MFR Murata -> (none); MOUNT 0603 -> (none); PKG (none) -> 0603
- C57: renamed from C52; DIGIKEY (none) -> 490-3285-1-ND; DKPN 490-3285-1-ND -> (none); LCSC (none) -> C77058; LCSCPN C77058 -> (none); MFR Murata -> (none); MOUNT 0603 -> (none); PKG (none) -> 0603
- C58: renamed from C53; DKPN 399-6123-ND -> (none); MFR KEMET -> (none); MOUNT Radial -> (none); PKG (none) -> Radial
- C59: renamed from C54; DKPN 399-6123-ND -> (none); MFR KEMET -> (none); MOUNT Radial -> (none); PKG (none) -> Radial
- C6: renamed from C4; DKPN B41866D6108M000 -> (none); LCSC (none) -> C1650604; LCSCPN C1650604 -> (none); MFR TDK -> (none); MOUNT Radial -> (none); PKG (none) -> Radial
- C60: renamed from C55; DKPN 399-6123-ND -> (none); MFR KEMET -> (none); MOUNT Radial -> (none); PKG (none) -> Radial
- C7: renamed from C5; DKPN 490-12456-1-ND -> (none); LCSCPN C417124 -> (none); MFR Murata -> (none)
- C8: renamed from C6; DKPN 490-3285-1-ND -> (none); LCSCPN C77058 -> (none); MFR Murata -> (none); MOUNT 0603 -> (none); PKG (none) -> 0603
- C9: renamed from C30; DKPN 399-ESY476M050AE3AA-ND -> (none); MFR KEMET -> (none); MOUNT Radial -> (none); PKG (none) -> Radial
- D1: renamed from D3; DKPN SS34FSCT-ND -> (none); MFR Onsemi -> (none)
- D2: renamed from D1; DKPN SMBJ28A-FDICT-ND -> (none); MFR Diodes -> (none); MOUNT DO-214AA -> (none); PKG (none) -> DO-214AA
- D3: renamed from D2; DIGIKEY (none) -> BZT52C12S-FDICT-ND; DKPN BZT52C12S-FDICT-ND -> (none); LCSC (none) -> C124208; MFR Diodes -> (none); PKG (none) -> SOD-323
- D4: DKPN SS34FSCT-ND -> (none); MFR Onsemi -> (none)
- DC1: DKPN 1866-3321-ND -> (none); MFR MEAN WELL USA Inc. -> (none)
- F1: DKPN F2589CT-ND -> (none); MFR Littelfuse -> (none)
- FB1: DKPN 490-13269-1-ND -> (none); MFR Murata -> (none); MOUNT 1206 -> (none); PKG (none) -> 1206
- FB2, FB3, FB4, FB5: DKPN 445-MPZ1608S600ATDH5CT-ND -> (none); MFR TDK -> (none); MPN MPZ1608S600ATDH5 -> (none)
- H1: renamed from H9; DKPN WM7624CT-ND -> (none); MFR Molex -> (none); MPN 0532610671 -> (none)
- H2: renamed from H1; DKPN 277-1106-ND -> (none); MFR Phoenix Contact -> (none)
- H3: DIGIKEY (none) -> 277-6377-ND; DKPN 277-6377-ND -> (none); LCSC (none) -> C5355140; MFR Phoenix Contact -> (none); SERIES (none) -> COMBICON MC
- H4: renamed from H5; DIGIKEY (none) -> 277-6377-ND; DKPN 277-6377-ND -> (none); LCSC (none) -> C5355140; MFR Phoenix Contact -> (none); SERIES (none) -> COMBICON MC
- H5: renamed from H2; DIGIKEY (none) -> 455-1721-ND; DKPN 455-1721-ND -> (none); LCSC (none) -> C157926; MFR JST -> (none); SERIES (none) -> PH
- H6: renamed from H4; DIGIKEY (none) -> 455-1721-ND; DKPN 455-1721-ND -> (none); LCSC (none) -> C157926; MFR JST -> (none); SERIES (none) -> PH
- H7: renamed from H6; DIGIKEY (none) -> 455-2243-ND; DKPN 455-2243-ND -> (none); LCSC (none) -> C157925; MFR JST -> (none); SERIES (none) -> XH
- H8: renamed from H7; DIGIKEY (none) -> 455-2243-ND; DKPN 455-2243-ND -> (none); LCSC (none) -> C157925; MFR JST -> (none); SERIES (none) -> XH
- H9: renamed from H8; DIGIKEY (none) -> 455-2243-ND; DKPN 455-2243-ND -> (none); LCSC (none) -> C157925; MFR JST -> (none); SERIES (none) -> XH
- J1: DIGIKEY (none) -> 2223-TB0011-350-04BE-ND; DKPN 2223-TB0011-350-04BE-ND -> (none); MFR Same Sky -> (none)
- J2: renamed from J3; DKPN A32259-ND -> (none); MANUFACTURER TE Connectivity -> (none); MFR TE Connectivity -> (none); SLSC C5166169 -> (none); STANDARD Manufacturer Recommendations -> (none)
- J3: renamed from J4; DKPN A32259-ND -> (none); MANUFACTURER TE Connectivity -> (none); MFR TE Connectivity -> (none); SLSC C5166169 -> (none); STANDARD Manufacturer Recommendations -> (none)
- J4: renamed from J5; DKPN A32259-ND -> (none); MANUFACTURER TE Connectivity -> (none); MFR TE Connectivity -> (none); SLSC C5166169 -> (none); STANDARD Manufacturer Recommendations -> (none)
- L1: DKPN SDR1307-100MLCT-ND -> (none); MFR Bourns -> (none)
- M1: DKPN ESP32-C6-DEVKITC-1-N8 -> (none); MFR Espressif Systems -> (none)
- M2: DKPN 5016-EZO-PH-ND -> (none); MFR Atlas Scientific -> (none)
- M3: DKPN 5016-EZO-EC-ND -> (none); MFR Atlas Scientific -> (none)
- M4: DKPN 5016-EZO-RTD-ND -> (none); MFR Atlas Scientific -> (none)
- P1: renamed from P13; DKPN WM1724-ND -> (none); MFR Molex -> (none); MPN 0510210600 -> (none)
- P2: renamed from P1; DKPN 277-1011-ND -> (none); MFR Phoenix Contact -> (none)
- P3: DIGIKEY (none) -> 277-6146-ND; DKPN 277-6146-ND -> (none); MFR Phoenix Connect -> (none)
- P4: renamed from P6; DIGIKEY (none) -> 277-6146-ND; DKPN 277-6146-ND -> (none); MFR Phoenix Connect -> (none)
- P5: renamed from P2; DIGIKEY (none) -> 455-1164-ND; DKPN 455-1164-ND -> (none); MFR JST -> (none)
- P6: renamed from P5; DIGIKEY (none) -> 455-1164-ND; DKPN 455-1164-ND -> (none); MFR JST -> (none)
- P7, P8, P9: DIGIKEY (none) -> 455-2267-ND; DKPN 455-2267-ND -> (none); LCSC (none) -> C144403; MFR JST -> (none); SERIES (none) -> XH
- PR1: MFR Benewake -> (none)
- PR2: renamed from PR3; DKPN 4152-ENV-40-PH-ND -> (none); MFR Bluelab -> (none)
- PR3: renamed from PR4; MFR Bluelab -> (none)
- PR4: renamed from PR5; DKPN 5016-PT-1000-ND -> (none); MFR Atlas Scientific -> (none)
- PR6: DKPN 4152-ENV-40-PH-ND -> (none)
- R1: renamed from R8; DKPN 311-100CRCT-ND -> (none); MFR Yageo -> (none); MGR Yageo -> (none)
- R10: renamed from R21; DKPN 311-100CRCT-ND -> (none); MGR Yageo -> (none)
- R11: renamed from R22; DKPN 311-4.70KCRCT-ND -> (none); MFR Yageo -> (none)
- R12: renamed from R23; DKPN 311-10.0KCRCT-ND -> (none); MFR Yageo -> (none)
- R13: renamed from R7; DKPN 311-21.0KCRCT-ND -> (none); MFR Yageo -> (none)
- R14: renamed from R11; DKPN 311-52.3KCRCT-ND -> (none); MFR Yageo -> (none)
- R15: renamed from R12; DKPN 311-10.0KCRCT-ND -> (none); MFR Yageo -> (none)
- R16: renamed from R13; DKPN 311-2.20KCRCT-ND -> (none); MFR Yageo -> (none)
- R17: renamed from R14; DKPN 311-2.20KCRCT-ND -> (none); MFR Yageo -> (none)
- R18: renamed from R15; DKPN 311-2.20KCRCT-ND -> (none); MFR Yageo -> (none)
- R19: renamed from R16; DKPN 311-2.20KCRCT-ND -> (none); MFR Yageo -> (none)
- R2: renamed from R9; DKPN 311-4.70KCRCT-ND -> (none); MFR Yageo -> (none)
- R20: renamed from R17; DKPN 311-16.9KCRCT-ND -> (none); MFR Yageo -> (none)
- R21: renamed from R18; DKPN 311-16.9KCRCT-ND -> (none); MFR Yageo -> (none)
- R22: renamed from R19; DKPN 311-10.0KCRCT-ND -> (none); MFR Yageo -> (none)
- R23: renamed from R20; DKPN 311-10.0KCRCT-ND -> (none); MFR Yageo -> (none)
- R24: renamed from R27; DKPN 13-RC0805FR-1014KLCT-ND -> (none); MFR Yageo -> (none)
- R25: renamed from R28; DKPN 311-10.7KCRCT-ND -> (none); MFR Yageo -> (none)
- R26: renamed from R29; DKPN 13-RC0805FR-1014KLCT-ND -> (none); MFR Yageo -> (none)
- R27: renamed from R30; DKPN 311-10.7KCRCT-ND -> (none); MFR Yageo -> (none)
- R28: renamed from R31; DKPN 13-RC0805FR-1014KLCT-ND -> (none); MFR Yageo -> (none)
- R29: renamed from R32; DKPN 311-10.7KCRCT-ND -> (none); MFR Yageo -> (none)
- R3: renamed from R1; DKPN 311-2.20KCRCT-ND -> (none); MFR Yageo -> (none)
- R34: renamed from R24; DIGIKEY (none) -> RL12S.11FCT-ND; DKPN RL12S.11FCT-ND -> (none); MFR Susumu -> (none)
- R35: renamed from R33; DIGIKEY (none) -> RL12S.11FCT-ND; DKPN RL12S.11FCT-ND -> (none); MFR Susumu -> (none)
- R4: renamed from R2; DKPN 311-2.20KCRCT-ND -> (none); MFR Yageo -> (none)
- R5: renamed from R10; DKPN 311-10.0KCRCT-ND -> (none); MFR Yageo -> (none)
- R6: renamed from R3; DKPN 311-10.0KCRCT-ND -> (none); MFR Yageo -> (none)
- R7: renamed from R4; DKPN 13-RC0805FR-1333KLCT-ND -> (none); MFR Yageo -> (none); MOUNT 0805 -> (none); PKG (none) -> 0805
- R8: renamed from R5; DKPN 311-1.00KCRCT-ND -> (none); MFR Yageo -> (none)
- R9: renamed from R6; DKPN 311-10.0KCRCT-ND -> (none); MFR Yageo -> (none)
- T1: renamed from T2; DIGIKEY (none) -> MMBT3904LT1GOSCT-ND; DKPN MMBT3904LT1GOSCT-ND -> (none); LCSC (none) -> C81464; MFR Onsemi -> (none); O Onsemi -> (none)
- T2: renamed from T3; DIGIKEY (none) -> IRLR2905PBFCT-ND; DKPN IRLR2905PBFCT-ND -> (none); LCSC (none) -> C3010; MFR Infineon -> (none); PKG (none) -> TO-252AA (DPAK)
- T3: renamed from T1; DKPN 785-1421-1-ND -> (none); MFR Alpha & Omega -> (none); MOUNT 8-DFN (5x6) -> (none); PKG (none) -> 8-DFN (5x6)
- T4: DIGIKEY (none) -> MMBT3904LT1GOSCT-ND; DKPN MMBT3904LT1GOSCT-ND -> (none); LCSC (none) -> C81464; MFR Onsemi -> (none); O Onsemi -> (none)
- T5: DKPN 785-1000-1-ND -> (none); MFR Alpha & Omega -> (none)
- U1: DIGIKEY (none) -> 296-TPS62933DRLRCT-ND; DKPN 296-TPS62933DRLRCT-ND -> (none); MFR Texas Instruments -> (none)
- U2: DKPN AZ1117IH-3.3TRG1DICT-ND -> (none); MFR Diodes -> (none)
- U3, U4: DKPN 505-ADM3260ARSZ-ND -> (none); MFR Analog Devices -> (none)
- U5, U6, U7: DIGIKEY (none) -> 175-TMC2209-LA-TCT-ND; DKPN 175-TMC2209-LA-TCT-ND -> (none); MFR Analog Devices -> (none)
- renumbered PR2 to PR5, P4 to PUMP1, P10 to PUMP2, P11 to PUMP3, P12 to PUMP4
Connections:
- net BRA_{NA}: now also R30.1
- net BRA_{NB}: now also R32.1
- net BRB_{NA}: now also R31.1
- net BRB_{NB}: now also R33.1
- net GND: now also R30.2, R31.2, R32.2, R33.2
