File: media/schematics/ATO-Valve.kicad_sch (KiCad schematic)
At the start: 11 parts

Commit message: update
Parts:
- removed H: MC_0.15", Coert-Vonk:TERM BLK HDR 2POS 3.81mm, symbol Coert-Vonk:TERM BLK HDR 2POS MC 3.81mm
- removed P: MC_0.15", Coert-Vonk:TERM BLOCK PLUG 2POS 3.81mm 1803578, symbol Coert-Vonk:TERM BLK PLG 2POS MC 3.81mm
- added HDR: MC_0.2", Coert-Vonk:TERM BLK HDR 2POS 5.08mm, symbol Coert-Vonk:TERM BLK HDR 2POS PC-MC 0.2{dblquote}
- added PLG: MC_0.2", Coert-Vonk:TERM BLK PLG 2POS PC-MC 0.2, symbol Coert-Vonk:TERM BLK PLG 2POS PC-MC 0.2{dblquote}
- renumbered C_{blk} to C_{b}, R_{dn} to R_{l}
Connections:
- net 24V: now also HDR.1
- net at D.A, N-CH.3 (D): now also HDR.2
- net at VALVE.24V: now also PLG.1
- net at VALVE.GND: now also PLG.2
Changed lines of the file:
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@@
 		(on_board yes)
 		(dnp no)
-		(property "Reference" "C_{blk}"
+		(property "Reference" "C_{b}"
 			(at 101.6 51.054 0)
 			(effects
@@
 			(project ""
 				(path "/a0000000-0000-4000-8000-000000002687"
-					(reference "C_{blk}")
+					(reference "C_{b}")
 					(unit 1)
 				)
@@
 	)
 	(symbol
-		(lib_id "Coert-Vonk:TERM BLK PLG 2POS MC 3.81mm")
-		(at 129.54 54.61 0)
-		(mirror y)
-		(unit 1)
-		(exclude_from_sim no)
-		(in_bom yes)
-		(on_board no)
-		(dnp no)
-		(property "Reference" "P"
-			(at 129.54 64.262 0)
-			(effects
-				(font
-					(size 1.27 1.27)
-				)
-			)
-		)
-		(property "Value" "MC_0.15\""
-			(at 129.54 66.548 0)
-			(effects
-				(font
-					(size 1.27 1.27)
-				)
-				(hide yes)
-			)
-		)
-		(property "Footprint" "Coert-Vonk:TERM BLOCK PLUG 2POS 3.81mm 1803578"
-			(at 129.54 54.61 0)
-			(effects
-				(font
-					(size 1.27 1.27)
-					(italic yes)
-				)
-				(hide yes)
-			)
-		)
-		(property "Datasheet" "https://mm.digikey.com/Volume0/opasdata/d220001/medias/docus/2411/1840zzz%2C%201803zzz.pdf"
-			(at 129.54 54.61 0)
-			(effects
-				(font
-					(size 1.27 1.27)
-					(italic yes)
-				)
-				(hide yes)
-			)
-		)
-		(property "Description" "2 Position Terminal Block Plug, Female Sockets 0.150\" (3.81mm) 180° Free Hanging (In-Line)"
-			(at 129.54 54.61 0)
-			(effects
-				(font
-					(size 1.27 1.27)
-				)
-				(hide yes)
-			)
-		)
-		(property "DKPN" "277-1161-ND"
-			(at 129.54 54.61 0)
-			(effects
-				(font
-					(size 1.27 1.27)
-				)
-				(hide yes)
-			)
-		)
-		(property "MFR" "Phoenix Connect"
-			(at 129.54 54.61 0)
-			(effects
-				(font
-					(size 1.27 1.27)
-				)
-				(hide yes)
-			)
-		)
-		(property "MPN" "1803578"
-			(at 129.54 54.61 0)
-			(effects
-				(font
-					(size 1.27 1.27)
-				)
-				(hide yes)
-			)
-		)
-		(pin "1"
-		)
-		(pin "2"
-		)
-		(instances
-			(project ""
-				(path "/a0000000-0000-4000-8000-000000002687"
-					(reference "P")
-					(unit 1)
-				)
-			)
-		)
-	)
-	(symbol
 		(lib_id "Coert-Vonk:CAP X7R 100nF ±10% 50V 0402 Murata")
 		(at 105.41 58.42 270)
@@
 	)
 	(symbol
+		(lib_id "Coert-Vonk:TERM BLK HDR 2POS PC-MC 0.2{dblquote}")
+		(at 125.73 54.61 0)
+		(mirror y)
+		(unit 1)
+		(exclude_from_sim no)
+		(in_bom yes)
+		(on_board yes)
+		(dnp no)
+		(property "Reference" "HDR"
+			(at 123.19 52.324 0)
+			(effects
+				(font
+					(size 1.27 1.27)
+				)
+			)
+		)
+		(property "Value" "MC_0.2\""
+			(at 123.19 52.07 0)
+			(effects
+				(font
+					(size 1.27 1.27)
+				)
+				(hide yes)
+			)
+		)
+		(property "Footprint" "Coert-Vonk:TERM BLK HDR 2POS 5.08mm"
+			(at 128.27 72.136 0)
+			(effects
+				(font
+					(size 0.762 0.762)
+				)
+				(hide yes)
+			)
+		)
+		(property "Datasheet" "https://www.phoenixcontact.com/us/products/1836189/pdf"
+			(at 130.81 54.61 0)
+			(effects
+				(font
+					(size 1.27 1.27)
+				)
+				(hide yes)
+			)
+		)
+		(property "Description" "2 Position Terminal Block Header, Male Pins, Shrouded (4 Side) 0.200\" (5.08mm) 90°, Right Angle Through Hole"
+			(at 127.508 63.5 0)
+			(effects
+				(font
+					(size 0.762 0.762)
+				)
+				(hide yes)
+			)
+		)
+		(property "DKPN" "277-6377-ND"
+			(at 125.73 54.61 0)
+			(effects
+				(font
+					(size 1.27 1.27)
+				)
+				(hide yes)
+			)
+		)
+		(property "MFR" "Phoenix Contact"
+			(at 125.73 54.61 0)
+			(effects
+				(font
+					(size 1.27 1.27)
+				)
+				(hide yes)
+			)
+		)
+		(property "PN" "1836189"
+			(at 125.73 54.61 0)
+			(effects
+				(font
+					(size 1.27 1.27)
+				)
+				(hide yes)
+			)
+		)
+		(pin "1"
+		)
+		(pin "2"
+		)
+		(instances
+			(project "ATO-Valve"
+				(path "/a0000000-0000-4000-8000-000000002687"
+					(reference "HDR")
+					(unit 1)
+				)
+			)
+		)
+	)
+	(symbol
 		(lib_id "Coert-Vonk:TRANS NPN 40V 0.2A SOT23-3")
 		(at 99.06 82.55 0)
@@
 	)
 	(symbol
-		(lib_id "Coert-Vonk:TERM BLK HDR 2POS MC 3.81mm")
-		(at 125.73 54.61 0)
+		(lib_id "Coert-Vonk:TERM BLK PLG 2POS PC-MC 0.2{dblquote}")
+		(at 129.54 54.61 0)
 		(mirror y)
 		(unit 1)
 		(exclude_from_sim no)
 		(in_bom yes)
-		(on_board yes)
-		(dnp no)
-		(property "Reference" "H"
-			(at 123.19 52.578 0)
-			(effects
-				(font
-					(size 1.27 1.27)
-				)
-			)
-		)
-		(property "Value" "MC_0.15\""
-			(at 122.682 52.578 0)
-			(effects
-				(font
-					(size 1.27 1.27)
-				)
-				(hide yes)
-			)
-		)
-		(property "Footprint" "Coert-Vonk:TERM BLK HDR 2POS 3.81mm"
-			(at 128.27 72.136 0)
-			(effects
-				(font
-					(size 0.762 0.762)
-				)
-				(hide yes)
-			)
-		)
-		(property "Datasheet" "https://www.phoenixcontact.com/us/products/1803277/pdf"
-			(at 130.81 54.61 0)
-			(effects
-				(font
-					(size 1.27 1.27)
-				)
-				(hide yes)
-			)
-		)
-		(property "Description" "2 Position Terminal Block Header, Male Pins, Shrouded (4 Side) 0.150\" (3.81mm) 90°, Right Angle Through Hole"
-			(at 127.508 63.5 0)
-			(effects
-				(font
-					(size 0.762 0.762)
-				)
-				(hide yes)
-			)
-		)
-		(property "DKPN" "277-1206-ND"
-			(at 125.73 54.61 0)
+		(on_board no)
+		(dnp no)
+		(property "Reference" "PLG"
+			(at 129.286 52.324 0)
+			(effects
+				(font
+					(size 1.27 1.27)
+				)
+			)
+		)
+		(property "Value" "MC_0.2\""
+			(at 129.54 67.31 0)
+			(effects
+				(font
+					(size 1.27 1.27)
+				)
+				(hide yes)
+			)
+		)
+		(property "Footprint" "Coert-Vonk:TERM BLK PLG 2POS PC-MC 0.2"
+			(at 129.54 54.61 0)
+			(effects
+				(font
+					(size 1.27 1.27)
+					(italic yes)
+				)
+				(hide yes)
+			)
+		)
+		(property "Datasheet" "https://mm.digikey.com/Volume0/opasdata/d220001/medias/docus/540/1836079.pdf"
+			(at 129.54 54.61 0)
+			(effects
+				(font
+					(size 1.27 1.27)
+					(italic yes)
+				)
+				(hide yes)
+			)
+		)
+		(property "Description" "2 Position Terminal Block Plug, Female Sockets 0.200\" (5.08mm) 180° Free Hanging (In-Line)"
+			(at 129.54 54.61 0)
+			(effects
+				(font
+					(size 1.27 1.27)
+				)
+				(hide yes)
+			)
+		)
+		(property "DKPN" "277-6146-ND"
+			(at 129.54 54.61 0)
 			(effects
 				(font
@@
 		)
 		(property "MFR" "Phoenix Connect"
-			(at 125.73 54.61 0)
-			(effects
-				(font
-					(size 1.27 1.27)
-				)
-				(hide yes)
-			)
-		)
-		(property "MPN" "1803277"
-			(at 125.73 54.61 0)
+			(at 129.54 54.61 0)
+			(effects
+				(font
+					(size 1.27 1.27)
+				)
+				(hide yes)
+			)
+		)
+		(property "PN" "1836079"
+			(at 129.54 54.61 0)
+			(effects
+				(font
+					(size 1.27 1.27)
+				)
+				(hide yes)
+			)
+		)
+		(property "SERIES" "MC"
+			(at 129.54 54.61 0)
 			(effects
 				(font
@@
 		)
 		(instances
-			(project ""
-				(path "/a0000000-0000-4000-8000-000000002687"
-					(reference "H")
+			(project "ATO-Valve"
+				(path "/a0000000-0000-4000-8000-000000002687"
+					(reference "PLG")
 					(unit 1)
 				)
@@
 		(on_board yes)
 		(dnp no)
-		(property "Reference" "R_{dn}"
+		(property "Reference" "R_{l}"
 			(at 108.458 82.296 90)
 			(effects
@@
 			(project "OPNhydro_r2"
 				(path "/a0000000-0000-4000-8000-000000002687"
-					(reference "R_{dn}")
-					(unit 1)
-				)
+					(reference "R_{l}")
+					(unit 1)
+				)
