File: media/schematics/ESP32-C6.kicad_sch (KiCad schematic)
At the start: 4 parts

Commit message: update
Parts:
- renumbered R_{up} to R_{h}
Other:
- moved on the sheet: MB
Changed lines of the file:
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@@
 	)
 	(no_connect
-		(at 154.94 46.99)
+		(at 148.59 46.99)
 	)
 	(no_connect
@@
 	(wire
 		(pts
-			(xy 134.62 46.99) (xy 133.35 46.99)
+			(xy 128.27 46.99) (xy 127 46.99)
 		)
 		(stroke
@@
 	(wire
 		(pts
-			(xy 144.78 57.15) (xy 144.78 58.42)
+			(xy 138.43 57.15) (xy 138.43 58.42)
 		)
 		(stroke
@@
 	(wire
 		(pts
-			(xy 133.35 39.37) (xy 133.35 46.99)
+			(xy 127 41.91) (xy 127 46.99)
 		)
 		(stroke
@@
 		(length 2.54)
 		(shape round)
-		(at 133.35 46.99 90)
+		(at 127 46.99 90)
 		(fields_autoplaced yes)
 		(effects
@@
 		)
 		(property "Netclass" "Power"
-			(at 130.81 46.2915 90)
+			(at 124.46 46.2915 90)
 			(effects
 				(font
@@
 		)
 		(property "Component Class" ""
-			(at -82.55 11.43 0)
+			(at -88.9 11.43 0)
 			(effects
 				(font
@@
 	(symbol
 		(lib_id "Coert-Vonk:GND")
-		(at 144.78 58.42 0)
+		(at 138.43 58.42 0)
 		(unit 1)
 		(exclude_from_sim no)
@@
 		(dnp no)
 		(property "Reference" "#PWR51"
-			(at 144.78 64.77 0)
+			(at 138.43 64.77 0)
 			(effects
 				(font
@@
 		)
 		(property "Value" "GND"
-			(at 144.78 62.23 0)
+			(at 138.43 62.23 0)
 			(effects
 				(font
@@
 		)
 		(property "Footprint" ""
-			(at 144.78 58.42 0)
+			(at 138.43 58.42 0)
 			(effects
 				(font
@@
 		)
 		(property "Datasheet" ""
-			(at 144.78 58.42 0)
+			(at 138.43 58.42 0)
 			(effects
 				(font
@@
 		)
 		(property "Description" "Power symbol creates a global label with name \"GND\" , ground"
-			(at 144.78 58.42 0)
+			(at 138.43 58.42 0)
 			(effects
 				(font
@@
 		(on_board yes)
 		(dnp no)
-		(property "Reference" "R_{up}"
+		(property "Reference" "R_{h}"
 			(at 53.34 48.006 90)
 			(effects
@@
 			(project "OPNhydro_r2"
 				(path "/a0000000-0000-4000-8000-000000002687"
-					(reference "R_{up}")
+					(reference "R_{h}")
 					(unit 1)
 				)
@@
 	(symbol
 		(lib_id "Coert-Vonk:EVAL ESP32-C6-DEVKITC-1-N8")
-		(at 139.7 44.45 0)
+		(at 133.35 44.45 0)
 		(unit 2)
 		(exclude_from_sim no)
@@
 		(dnp no)
 		(property "Reference" "M"
-			(at 144.78 41.91 0)
+			(at 138.43 41.91 0)
 			(effects
 				(font
@@
 		)
 		(property "Value" "ESP32-C6-DEVKIT"
-			(at 144.78 41.91 0)
+			(at 138.43 41.91 0)
 			(effects
 				(font
@@
 		)
 		(property "Footprint" "Coert-Vonk:EVAL ESP32-C6-DEVKITC"
-			(at 139.7 44.45 0)
+			(at 133.35 44.45 0)
 			(effects
 				(font
@@
 		)
 		(property "Datasheet" "https://mm.digikey.com/Volume0/opasdata/d220001/medias/docus/5528/ESP32-C6-DEVKITC-1-N8.pdf"
-			(at 139.7 44.45 0)
+			(at 133.35 44.45 0)
 			(effects
 				(font
@@
 		)
 		(property "Description" "The ESP32-C6-DEVKITC-1-N8 from Espressif Systems is a development board designed for RF, RFID, and wireless applications. Built around the ESP32-C6-WROOM-1 module, it supports multiple connectivity options including 802.11 b/g/n/ax Wi-Fi, Bluetooth® (BLE), and 802.15.4 for Thread and Zigbee® protocols. The board is powered by the ESP32-C6 chip with 8MB SPI flash, offering advanced processing power and efficient memory management. It features GPIO ports for extensive interfacing, along with a USB Type-C™ to UART port for power and communication. The board also includes a USB-to-UART bridge, pin header, and boot/reset buttons, operating at 3.3V with a 5V to 3.3V power regulator. This development board is ideal for exploring a wide range of wireless applications, including IoT, smart home devices, and RF communication projects."
-			(at 139.7 44.45 0)
+			(at 133.35 44.45 0)
 			(effects
 				(font
@@
 		)
 		(property "DKPN" "ESP32-C6-DEVKITC-1-N8"
-			(at 139.7 44.45 0)
+			(at 133.35 44.45 0)
 			(effects
 				(font
@@
 	(symbol
 		(lib_id "power:+5V")
-		(at 133.35 39.37 0)
+		(at 127 41.91 0)
 		(unit 1)
 		(exclude_from_sim no)
@@
 		(dnp no)
 		(property "Reference" "#PWR049"
-			(at 133.35 43.18 0)
+			(at 127 45.72 0)
 			(effects
 				(font
@@
 		)
 		(property "Value" "5V"
-			(at 133.35 35.306 0)
+			(at 127 37.846 0)
 			(effects
 				(font
@@
 		)
 		(property "Footprint" ""
-			(at 133.35 39.37 0)
+			(at 127 41.91 0)
 			(effects
 				(font
@@
 		)
 		(property "Datasheet" ""
-			(at 133.35 39.37 0)
+			(at 127 41.91 0)
 			(effects
 				(font
@@
 		)
 		(property "Description" "Power symbol creates a global label with name \"+5V\""
-			(at 133.35 39.37 0)
+			(at 127 41.91 0)
 			(effects
 				(font
@@
 		(on_board yes)
 		(dnp no)
-		(property "Reference" "R_{up}"
+		(property "Reference" "R_{h}"
 			(at 63.246 48.006 90)
 			(effects
@@
 			(project ""
 				(path "/a0000000-0000-4000-8000-000000002687"
-					(reference "R_{up}")
+					(reference "R_{h}")
 					(unit 1)
 				)
