File: media/schematics/Float-Switches.kicad_sch (KiCad schematic)
At the start: 7 parts, among them SW1 FLOAT, SW2 FLOAT

Commit message: update
Parts:
- removed J: MKDS, Coert-Vonk:TERM BLK 4POS SCREW 3.5mm, symbol Coert-Vonk:TERM BLK SCREW 4POS MKDS 3.5mm
- added J: SS-3.5mm, Coert-Vonk:TERM BLK 4POS SCREW 3.5mm, symbol Coert-Vonk:TERM BLK SCREW 4POS SS-MKDS 3.5mm
- renumbered C_{fh} to C, C_{fl} to C, R_{fl} to R, R_{fh} to R
Connections:
- net 3V3: now also J.1 (Pin_1)
- net FLOAT_HIGH: now also J.2 (Pin_2)
- net FLOAT_LOW: now also J.3 (Pin_3)
- net GND: now also J.4 (Pin_4)
Other:
- moved on the sheet: C, R
