File: media/schematics/LiDAR.kicad_sch (KiCad schematic)
At the start: 4 parts

Commit message: update
Parts:
- renumbered C_{blk} to C_{b}, H to HDR, P to PLG
Changed lines of the file:
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@@
 		(on_board yes)
 		(dnp no)
-		(property "Reference" "H"
-			(at 105.41 58.674 0)
+		(property "Reference" "HDR"
+			(at 106.172 58.674 0)
 			(effects
 				(font
@@
 			(project ""
 				(path "/a0000000-0000-4000-8000-000000002687"
-					(reference "H")
+					(reference "HDR")
 					(unit 1)
 				)
@@
 		(on_board yes)
 		(dnp no)
-		(property "Reference" "C_{blk}"
+		(property "Reference" "C_{b}"
 			(at 117.856 73.66 0)
 			(effects
@@
 			(project ""
 				(path "/a0000000-0000-4000-8000-000000002687"
-					(reference "C_{blk}")
+					(reference "C_{b}")
 					(unit 1)
 				)
@@
 		(on_board yes)
 		(dnp no)
-		(property "Reference" "P"
-			(at 101.6 81.026 0)
+		(property "Reference" "PLG"
+			(at 100.838 58.674 0)
 			(effects
 				(font
@@
 			(project ""
 				(path "/a0000000-0000-4000-8000-000000002687"
-					(reference "P")
+					(reference "PLG")
 					(unit 1)
 				)
