File: media/schematics/Linear-Regulator.kicad_sch (KiCad schematic)
At the start: 2 parts

Commit message: update
Parts:
- added C_{b1}: 22μF, Coert-Vonk:CAP X7R 22μF ±10 10V 1206, symbol Coert-Vonk:CAP X7R 22μF ±10% 10V 1206 Murata GRM
- renumbered C_{blk} to C_{b2}
Connections:
- net 5V: now also C_{b1}.2
- net GND: now also C_{b1}.1
Other:
- moved on the sheet: C_{b2}, U
