File: media/schematics/Main-Pump.kicad_sch (KiCad schematic)
At the start: 11 parts, among them T3 N-CH

Commit message: update
Parts:
- renumbered C_{blk} to C_{b}, H to HDR, P to PLG, R_{up} to R_{h}
Changed lines of the file:
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@@
 		(on_board yes)
 		(dnp no)
-		(property "Reference" "R_{up}"
+		(property "Reference" "R_{h}"
 			(at 104.648 71.12 90)
 			(effects
@@
 			(project ""
 				(path "/a0000000-0000-4000-8000-000000002687"
-					(reference "R_{up}")
+					(reference "R_{h}")
 					(unit 1)
 				)
@@
 		(on_board yes)
 		(dnp no)
-		(property "Reference" "H"
+		(property "Reference" "HDR"
 			(at 120.65 46.736 0)
 			(effects
@@
 			(project ""
 				(path "/a0000000-0000-4000-8000-000000002687"
-					(reference "H")
+					(reference "HDR")
 					(unit 1)
 				)
@@
 		(on_board no)
 		(dnp no)
-		(property "Reference" "P"
+		(property "Reference" "PLG"
 			(at 127 59.182 0)
 			(effects
@@
 			(project ""
 				(path "/a0000000-0000-4000-8000-000000002687"
-					(reference "P")
+					(reference "PLG")
 					(unit 1)
 				)
@@
 		(on_board yes)
 		(dnp no)
-		(property "Reference" "C_{blk}"
+		(property "Reference" "C_{b}"
 			(at 98.806 45.72 0)
 			(effects
@@
 			(project "OPNhydro_r2"
 				(path "/a0000000-0000-4000-8000-000000002687"
-					(reference "C_{blk}")
+					(reference "C_{b}")
 					(unit 1)
 				)
