File: media/schematics/Optional-I2C.kicad_sch (KiCad schematic)
At the start: 10 parts

Commit message: update
Parts:
- renumbered C_{blk} to C_{b}, H to HDR, P to PLG
Changed lines of the file:
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@@
 		(dnp no)
 		(property "Reference" "C_{mf}"
-			(at 80.264 71.882 90)
+			(at 80.772 71.882 90)
 			(effects
 				(font
@@
 		(on_board yes)
 		(dnp no)
-		(property "Reference" "H"
-			(at 71.12 56.642 0)
+		(property "Reference" "HDR"
+			(at 71.12 57.658 0)
 			(effects
 				(font
@@
 			(project ""
 				(path "/a0000000-0000-4000-8000-000000002687"
-					(reference "H")
+					(reference "HDR")
 					(unit 1)
 				)
@@
 		(on_board yes)
 		(dnp no)
-		(property "Reference" "H"
-			(at 125.73 56.642 0)
+		(property "Reference" "HDR"
+			(at 125.73 57.658 0)
 			(effects
 				(font
@@
 			(project "OPNhydro_r2"
 				(path "/a0000000-0000-4000-8000-000000002687"
-					(reference "H")
+					(reference "HDR")
 					(unit 1)
 				)
@@
 		(on_board yes)
 		(dnp no)
-		(property "Reference" "C_{blk}"
-			(at 145.542 72.898 90)
+		(property "Reference" "C_{b}"
+			(at 143.764 71.882 90)
 			(effects
 				(font
@@
 			(project "OPNhydro_r2"
 				(path "/a0000000-0000-4000-8000-000000002687"
-					(reference "C_{blk}")
+					(reference "C_{b}")
 					(unit 1)
 				)
@@
 		(on_board no)
 		(dnp yes)
-		(property "Reference" "P"
+		(property "Reference" "PLG"
 			(at 65.024 74.676 0)
 			(effects
@@
 			(project ""
 				(path "/a0000000-0000-4000-8000-000000002687"
-					(reference "P")
+					(reference "PLG")
 					(unit 1)
 				)
@@
 		(dnp no)
 		(property "Reference" "C_{mf}"
-			(at 134.874 71.882 90)
+			(at 135.382 71.882 90)
 			(effects
 				(font
@@
 		(on_board yes)
 		(dnp no)
-		(property "Reference" "C_{blk}"
-			(at 90.932 72.898 90)
+		(property "Reference" "C_{b}"
+			(at 89.154 71.882 90)
 			(effects
 				(font
@@
 			(project "OPNhydro_r2"
 				(path "/a0000000-0000-4000-8000-000000002687"
-					(reference "C_{blk}")
+					(reference "C_{b}")
 					(unit 1)
 				)
@@
 		(on_board no)
 		(dnp yes)
-		(property "Reference" "P"
+		(property "Reference" "PLG"
 			(at 119.634 74.676 0)
 			(effects
@@
 			(project "OPNhydro_r1"
 				(path "/a0000000-0000-4000-8000-000000002687"
-					(reference "P")
-					(unit 1)
-				)
+					(reference "PLG")
+					(unit 1)
+				)
