File: media/schematics/Stepper-Driver.kicad_sch (KiCad schematic)
At the start: 15 parts

Commit message: update
Parts:
- renumbered C_{blk1} to C_{b1}, C_{blk2} to C_{b2}, H to HDR, P to PLG, R_{l} to R_{b}, R_{sense} to R_{s}, R_{h} to R_{t}
Changed lines of the file:
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@@
 		(on_board yes)
 		(dnp no)
-		(property "Reference" "R_{l}"
+		(property "Reference" "R_{b}"
 			(at 69.088 80.01 90)
 			(effects
@@
 			(project ""
 				(path "/a0000000-0000-4000-8000-000000002687"
-					(reference "R_{l}")
+					(reference "R_{b}")
 					(unit 1)
 				)
@@
 		(on_board yes)
 		(dnp no)
-		(property "Reference" "C_{blk1}"
+		(property "Reference" "C_{b1}"
 			(at 55.88 73.152 90)
 			(effects
@@
 			(project "OPNhydro_r2"
 				(path "/a0000000-0000-4000-8000-000000002687"
-					(reference "C_{blk1}")
+					(reference "C_{b1}")
 					(unit 1)
 				)
@@
 		(on_board yes)
 		(dnp no)
-		(property "Reference" "H"
+		(property "Reference" "HDR"
 			(at 141.986 61.976 0)
 			(effects
@@
 			(project ""
 				(path "/a0000000-0000-4000-8000-000000002687"
-					(reference "H")
+					(reference "HDR")
 					(unit 1)
 				)
@@
 		(on_board yes)
 		(dnp no)
-		(property "Reference" "R_{h}"
+		(property "Reference" "R_{t}"
 			(at 69.088 69.85 90)
 			(effects
@@
 			(project ""
 				(path "/a0000000-0000-4000-8000-000000002687"
-					(reference "R_{h}")
+					(reference "R_{t}")
 					(unit 1)
 				)
@@
 		(on_board yes)
 		(dnp no)
-		(property "Reference" "R_{sense}"
+		(property "Reference" "R_{s}"
 			(at 120.65 80.772 0)
 			(effects
@@
 			(project "OPNhydro_r2"
 				(path "/a0000000-0000-4000-8000-000000002687"
-					(reference "R_{sense}")
+					(reference "R_{s}")
 					(unit 1)
 				)
@@
 		(on_board no)
 		(dnp no)
-		(property "Reference" "P"
-			(at 148.59 79.502 0)
+		(property "Reference" "PLG"
+			(at 148.336 61.976 0)
 			(effects
 				(font
@@
 			(project ""
 				(path "/a0000000-0000-4000-8000-000000002687"
-					(reference "P")
+					(reference "PLG")
 					(unit 1)
 				)
@@
 		(on_board yes)
 		(dnp no)
-		(property "Reference" "R_{sense}"
+		(property "Reference" "R_{s}"
 			(at 120.65 68.072 0)
 			(effects
@@
 			(project ""
 				(path "/a0000000-0000-4000-8000-000000002687"
-					(reference "R_{sense}")
+					(reference "R_{s}")
 					(unit 1)
 				)
@@
 		(dnp no)
 		(fields_autoplaced yes)
-		(property "Reference" "C_{blk2}"
+		(property "Reference" "C_{b2}"
 			(at 133.35 52.7938 0)
 			(effects
@@
 			(project "OPNhydro_r2"
 				(path "/a0000000-0000-4000-8000-000000002687"
-					(reference "C_{blk2}")
-					(unit 1)
-				)
+					(reference "C_{b2}")
+					(unit 1)
+				)
