File: media/schematics/Buck-Converter.kicad_sch (KiCad schematic)
At the start: 15 parts

Commit message: update
Parts:
- removed C_{blk} (x2): 10μF, Coert-Vonk:CAP X5R 10μF ±10 16V 0805 Murata GRM, symbol Coert-Vonk:CAP X5R 10μF ±10% 16V 0805 Murata GRM
- removed C_{hf} (x2): 10nF, Coert-Vonk:CAP X7R 10nF ±10 16V 0402 Murata, symbol Coert-Vonk:CAP X7R 10nF ±10% 16V 0402 Murata
- removed C_{mf} (x4): 100nF, Coert-Vonk:CAP X7R 100nF ±10 50V 0402 Murata, symbol Coert-Vonk:CAP X7R 100nF ±10% 50V 0402 Murata
- removed FB (x2): 60Ω at 100MHz, symbol Coert-Vonk:FERRITE BEAD 20mΩ 60Ω 0603 TDK
- removed R_{h}: 16k9, Coert-Vonk:RES 0805 YAGEO, symbol Coert-Vonk:RES 16.9kΩ ±1% 1/8W 0805 Yageo
- removed R_{up} (x2): 2k2, Coert-Vonk:RES 0805 YAGEO, symbol Coert-Vonk:RES 2.2kΩ ±1% 1/8W 0805 Yageo
- removed U: ADM3260, Coert-Vonk:IC ISOLTR 2.5KV 2CH I2C 20SSOP ADM3260, symbol Coert-Vonk:IC ISOLTR 2.5KV 2CH I2C 20SSOP ADM3260
- added C_{blk1}: 10μF, Coert-Vonk:CAP X7R 10μF ±10 50V 1206 Murata GRT, symbol Coert-Vonk:CAP X7R 10μF ±10% 50V 1206 Murata GRT
- added C_{blk2} (x3): 10μF, Coert-Vonk:CAP X5R 10μF ±10 16V 0805 Murata GRM, symbol Coert-Vonk:CAP X5R 10μF ±10% 16V 0805 Murata GRM
- added C_{blk3}: 220μF, Coert-Vonk:CAP ALUM-POLY 220μF ±20 16V Panasonic, symbol Coert-Vonk:CAP ALUM-POLY 220μF ±20% 16V Panasonic
- added C_{bst}, C_{mf}: 100nF, Coert-Vonk:CAP X7R 100nF ±10 50V 0402 Murata, symbol Coert-Vonk:CAP X7R 100nF ±10% 50V 0402 Murata
- added C_{ss}: 33nF, Coert-Vonk:CAP X7R 33nF ±10 50V 0805 Kemet, symbol Coert-Vonk:CAP X7R 33nF ±10% 50V 0805 Kemet
- added L: 10µH, Coert-Vonk:IND 10µH 5.6A 21mΩ, symbol Coert-Vonk:IND 10µH 5.6A 21mΩ
- added R_{h}: 52k3, Coert-Vonk:RES 0805 YAGEO, symbol Coert-Vonk:RES 52.3kΩ ±1% 1/8W 0805 Yageo
- added R_{rt}: 21k, Coert-Vonk:RES 0805 YAGEO, symbol Coert-Vonk:RES 21kΩ ±1% 1/8W 0805 Yageo
- added U: TPS62933, Coert-Vonk:REG ADJ 3A BUCK TPS62933 SOT583, symbol Coert-Vonk:REG ADJ 3A BUCK TPS62933 SOT583
Connections:
- net SCL_{ISO} is gone; now on net GND: R_{l}.1
- net GND: now also C_{blk1}.1, C_{blk2}.1, C_{blk2}.1, C_{blk2}.1, C_{blk3}.2, C_{mf}.1, C_{ss}.1, R_{rt}.1, U.4 (GND)
- net 0V8: now reaches R_{l}.2
- net 0V8: now also R_{h}.1, U.8 (FB)
- new net: C_{bst}.2, L.1, U.5 (SW)
- new net: C_{bst}.1, U.6 (BST)
- new net: C_{ss}.2, U.7 (SS)
- new net: R_{rt}.2, U.1 (RT)
- new net 24V: C_{blk1}.2, C_{mf}.2, U.3 (VIN)
- new net 5V: C_{blk2}.2, C_{blk2}.2, C_{blk2}.2, C_{blk3}.1, L.2, R_{h}.2
- no-connect marks 0 -> 1
Other:
- title: OPNhydro ADM3260 -> OPNhydro

Commit message: update
Parts:
- renumbered C_{blk1} to C_{b1}, C_{blk2} to C_{b2}, C_{blk3} to C_{b3}, R_{l} to R_{b}, R_{h} to R_{t}
Other:
- moved on the sheet: C_{b1}, C_{mf}, C_{ss}

Commit message: update
Parts:
- removed C_{b3}: 220μF, Coert-Vonk:CAP ALUM-POLY 220μF ±20 16V Panasonic, symbol Coert-Vonk:CAP ALUM-POLY 220μF ±20% 16V Panasonic
- added C_{b2}: 1000μF, Coert-Vonk:CAP ALUM-ELEC 1000μF ±20 50V TDK, symbol Coert-Vonk:CAP ALUM-ELEC 1000μF ±20% 50V TDK
- renumbered C_{b2} to C_{mf2}
Connections:
- net 5V: now also C_{b2}.1
- net GND: now also C_{b2}.2
Changed lines of the file:
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@@
 		(on_board yes)
 		(dnp no)
-		(property "Reference" "C_{b2}"
+		(property "Reference" "C_{mf2}"
 			(at 188.722 47.498 90)
 			(effects
@@
 			(project "OPNhydro_r2"
 				(path "/a0000000-0000-4000-8000-000000002687"
-					(reference "C_{b2}")
+					(reference "C_{mf2}")
 					(unit 1)
 				)
@@
 	)
 	(symbol
+		(lib_id "Coert-Vonk:CAP ALUM-ELEC 1000μF ±20% 50V TDK")
+		(at 194.31 50.8 0)
+		(unit 1)
+		(exclude_from_sim no)
+		(in_bom yes)
+		(on_board yes)
+		(dnp no)
+		(property "Reference" "C_{b2}"
+			(at 195.834 47.752 0)
+			(effects
+				(font
+					(size 1.27 1.27)
+				)
+				(justify left)
+			)
+		)
+		(property "Value" "1000μF"
+			(at 197.612 48.514 0)
+			(effects
+				(font
+					(size 1.27 1.27)
+				)
+				(justify left)
+				(hide yes)
+			)
+		)
+		(property "Footprint" "Coert-Vonk:CAP ALUM-ELEC 1000μF ±20 50V TDK"
+			(at 194.31 50.8 0)
+			(effects
+				(font
+					(size 1.27 1.27)
+				)
+				(hide yes)
+			)
+		)
+		(property "Datasheet" "https://www.tdk-electronics.tdk.com/inf/20/30/db/aec/B41866.pdf?ref_disty=digikey"
+			(at 194.31 50.8 0)
+			(effects
+				(font
+					(size 1.27 1.27)
+				)
+				(hide yes)
+			)
+		)
+		(property "Description" "1000 µF 50 V Aluminum Electrolytic Capacitors Radial, Can 39mOhm @ 100kHz 5000 Hrs @ 125°C"
+			(at 194.31 50.8 0)
+			(effects
+				(font
+					(size 1.27 1.27)
+				)
+				(hide yes)
+			)
+		)
+		(property "DKPN" "B41866D6108M000"
+			(at 194.31 50.8 0)
+			(effects
+				(font
+					(size 1.27 1.27)
+				)
+				(hide yes)
+			)
+		)
+		(property "MFR" "TDK"
+			(at 194.31 50.8 0)
+			(effects
+				(font
+					(size 1.27 1.27)
+				)
+				(hide yes)
+			)
+		)
+		(property "PN" "B41866D6108M000"
+			(at 194.31 50.8 0)
+			(effects
+				(font
+					(size 1.27 1.27)
+				)
+				(hide yes)
+			)
+		)
+		(property "SERIES" "B41866"
+			(at 194.31 50.8 0)
+			(effects
+				(font
+					(size 1.27 1.27)
+				)
+				(hide yes)
+			)
+		)
+		(pin "1"
+		)
+		(pin "2"
+		)
+		(instances
+			(project "Buck-Converter"
+				(path "/a0000000-0000-4000-8000-000000002687"
+					(reference "C_{b2}")
+					(unit 1)
+				)
+			)
+		)
+	)
+	(symbol
 		(lib_id "Coert-Vonk:CAP X7R 100nF ±10% 50V 0402 Murata")
 		(at 154.94 41.91 90)
@@
 		(on_board yes)
 		(dnp no)
-		(property "Reference" "C_{b2}"
+		(property "Reference" "C_{mf2}"
 			(at 176.022 47.498 90)
 			(effects
@@
 			(project ""
 				(path "/a0000000-0000-4000-8000-000000002687"
-					(reference "C_{b2}")
+					(reference "C_{mf2}")
 					(unit 1)
 				)
@@
 	)
 	(symbol
-		(lib_id "Coert-Vonk:CAP ALUM-POLY 220μF ±20% 16V Panasonic")
-		(at 194.31 50.8 0)
-		(unit 1)
-		(exclude_from_sim no)
-		(in_bom yes)
-		(on_board yes)
-		(dnp no)
-		(fields_autoplaced yes)
-		(property "Reference" "C_{b3}"
-			(at 196.85 50.2538 0)
-			(effects
-				(font
-					(size 1.27 1.27)
-				)
-				(justify left)
-			)
-		)
-		(property "Value" "220μF"
-			(at 196.85 51.5238 0)
-			(effects
-				(font
-					(size 1.27 1.27)
-				)
-				(justify left)
-				(hide yes)
-			)
-		)
-		(property "Footprint" "Coert-Vonk:CAP ALUM-POLY 220μF ±20 16V Panasonic"
-			(at 194.31 50.8 0)
-			(effects
-				(font
-					(size 1.27 1.27)
-				)
-				(hide yes)
-			)
-		)
-		(property "Datasheet" "https://industrial.panasonic.com/cdbs/www-data/pdf/AAB8000/AAB8000C226.pdf"
-			(at 194.31 50.8 0)
-			(effects
-				(font
-					(size 1.27 1.27)
-				)
-				(hide yes)
-			)
-		)
-		(property "Description" "220 µF 16 V Aluminum - Polymer Capacitors Radial, Can - SMD 22mOhm 1000 Hrs @ 125°C"
-			(at 194.31 50.8 0)
-			(effects
-				(font
-					(size 1.27 1.27)
-				)
-				(hide yes)
-			)
-		)
-		(property "DKPN" "P124158CT-ND"
-			(at 194.31 50.8 0)
-			(effects
-				(font
-					(size 1.27 1.27)
-				)
-				(hide yes)
-			)
-		)
-		(property "MFR" "Panasonic"
-			(at 194.31 50.8 0)
-			(effects
-				(font
-					(size 1.27 1.27)
-				)
-				(hide yes)
-			)
-		)
-		(property "PN" "16SVPK220M"
-			(at 194.31 50.8 0)
-			(effects
-				(font
-					(size 1.27 1.27)
-				)
-				(hide yes)
-			)
-		)
-		(pin "1"
-		)
-		(pin "2"
-		)
-		(instances
-			(project ""
-				(path "/a0000000-0000-4000-8000-000000002687"
-					(reference "C_{b3}")
-					(unit 1)
-				)
-			)
-		)
-	)
-	(symbol
 		(lib_id "Coert-Vonk:GND")
 		(at 167.64 62.23 0)
@@
 		(on_board yes)
 		(dnp no)
-		(property "Reference" "C_{b2}"
+		(property "Reference" "C_{mf2}"
 			(at 182.372 47.498 90)
 			(effects
@@
 			(project "OPNhydro_r2"
 				(path "/a0000000-0000-4000-8000-000000002687"
-					(reference "C_{b2}")
-					(unit 1)
-				)
+					(reference "C_{mf2}")
+					(unit 1)
+				)
