File: media/schematics/Isolation-Circuit.kicad_sch (KiCad schematic)
At the start: 15 parts

Commit message: update
Parts:
- renumbered R_{l} to R_{b}, R_{h} to R_{t}
Connections:
- net SCL_{ISO}: no longer R_{b}.1, R_{t}.1, R_{up}.1, U.13 (VSEL), U.18 (SDA_{1})
- new net: R_{b}.1, R_{t}.1, U.13 (VSEL)
- new net SDA_{ISO}: R_{up}.1, U.18 (SDA_{1})
Other:
- moved on the sheet: C_{blk}, C_{hf}, C_{mf}, FB, R_{b}, R_{t}, R_{up}

Commit message: update
Parts:
- renumbered C_{blk} to C_{b}
Changed lines of the file:
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@@
 		(on_board yes)
 		(dnp no)
-		(property "Reference" "C_{blk}"
+		(property "Reference" "C_{b}"
 			(at 133.858 52.324 90)
 			(effects
@@
 			(project "OPNhydro_r2"
 				(path "/a0000000-0000-4000-8000-000000002687"
-					(reference "C_{blk}")
+					(reference "C_{b}")
 					(unit 1)
 				)
@@
 		(on_board yes)
 		(dnp no)
-		(property "Reference" "C_{blk}"
+		(property "Reference" "C_{b}"
 			(at 80.772 52.324 90)
 			(effects
@@
 			(project "OPNhydro_r2"
 				(path "/a0000000-0000-4000-8000-000000002687"
-					(reference "C_{blk}")
+					(reference "C_{b}")
 					(unit 1)
 				)
