File: media/schematics/Protection-Gauntlet.kicad_sch (KiCad schematic)
At the start: 10 parts

Commit message: update
Parts:
- renumbered C_{blk} to C_{b}, H to HDR, P to PLG
Changed lines of the file:
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@@
 		(on_board yes)
 		(dnp no)
-		(property "Reference" "C_{blk}"
+		(property "Reference" "C_{b}"
 			(at 138.684 60.96 0)
 			(effects
@@
 			(project "Protection-Gauntlet"
 				(path "/a0000000-0000-4000-8000-000000002687"
-					(reference "C_{blk}")
+					(reference "C_{b}")
 					(unit 1)
 				)
@@
 		(on_board no)
 		(dnp no)
-		(property "Reference" "P"
-			(at 74.93 61.722 0)
+		(property "Reference" "PLG"
+			(at 74.93 49.53 0)
 			(effects
 				(font
@@
 			(project ""
 				(path "/a0000000-0000-4000-8000-000000002687"
-					(reference "P")
+					(reference "PLG")
 					(unit 1)
 				)
@@
 		(on_board yes)
 		(dnp no)
-		(property "Reference" "H"
+		(property "Reference" "HDR"
 			(at 81.28 49.53 0)
 			(effects
@@
 			(project "Protection-Gauntlet"
 				(path "/a0000000-0000-4000-8000-000000002687"
-					(reference "H")
-					(unit 1)
-				)
+					(reference "HDR")
+					(unit 1)
+				)
